File: hardware/om-god.kicad_pcb (KiCad board)
At the start: 4 copper layers, 536 parts, among them CN1 USB-B-Female-90, CN2 DIN-504B-M10, CN3 DIN-504B-M10, J1 Conn_01x13_Pin, J10 Conn_01x02_Socket, J11 Conn_01x08_Pin, J2 Conn_01x03_Pin, J3 PJ-625G, J4 PJ-625G, J5 PJ-625G, J6 Conn_01x08_Pin, J8 Conn_01x02_Socket, J9 Conn_01x02_Socket, Q1 Si7617DN, Q2 Si7617DN, Q3 Si7617DN, SW1 TS-1003ST-26, SW10 TS-1003ST-26, SW11 TS-1003ST-26, SW12 TS-1003ST-26, SW13 TS-1003ST-26, SW14 TS-1003ST-26, SW15 TS-1003ST-26, SW16 TS-1003ST-26, SW17 TS-1003ST-26, SW18 TS-1003ST-26, SW19 TS-1003ST-26, SW2 TS-1003ST-26, SW20 TS-1003ST-26, SW21 TS-1003ST-26, SW22 TS-1003ST-26, SW23 TS-1003ST-26, SW24 TS-1003ST-26, SW25 TS-1003ST-26, SW26 TS-1003ST-26, SW27 TS-1003ST-26, SW28 TS-1003ST-26, SW29 TS-1003ST-26, SW3 TS-1003ST-26, SW30 TS-1003ST-26, SW31 TS-1003ST-26, SW32 TS-1003ST-26, SW33 TS-1003ST-26, SW34 TS-1003ST-26, SW35 TS-1003ST-26, SW36 TS-1003ST-26, SW37 TS-1003ST-26, SW38 TS-1003ST-26, SW39 TS-1003ST-26, SW4 TS-1003ST-26, SW40 TS-1003ST-26, SW41 TS-1003ST-26, SW42 TS-1003ST-26, SW43 TS-1003ST-26, SW44 TS-1003ST-26, SW45 TS-1003ST-26, SW46 TS-1003ST-26, SW47 TS-1003ST-26, SW48 TS-1003ST-26, SW49 RotaryEncoder_Switch, SW5 TS-1003ST-26, SW50 RotaryEncoder, SW51 RotaryEncoder, SW52 RotaryEncoder, SW53 RotaryEncoder, SW54 RotaryEncoder, SW55 RotaryEncoder, SW56 TS-1003ST-26, SW57 TS-1003ST-26, SW58 TS-1003ST-26, SW59 SW_Push, SW6 TS-1003ST-26, SW60 SW_Push, SW7 TS-1003ST-26, SW8 TS-1003ST-26, SW9 TS-1003ST-26, U1 NE5532DR, U12 LMR33630ADDAR, U12 TPS55288RPMR, U13 LMR33630ADDAR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

Commit message: h
Parts:
- removed C135: 0.1uF, Capacitor_SMD:C_0402_1005Metric
- removed CN3: DIN-504B-M10, lcsc:CONN-TH_DIN-504B-M10
- removed D56, D57, D58, D59, D60, D61, D62, D63, D64, D65, D66, D67, D68, D69, D70, D71, D72: 1N4148WS_C917117, lcsc:SOD-323_L1.8-W1.3-LS2.5-RD
- removed R118: 0, Resistor_SMD:R_0402_1005Metric
- removed R119: 10k, Resistor_SMD:R_0402_1005Metric
- removed R120: 4.7k, Resistor_SMD:R_0402_1005Metric
- removed the U12 at (181.2, 129.8)
- removed the U12 at (213.4, 116.8)
- removed the U26 at (222.4, 65.8)
- removed the U26 at (46.6, 155.8)
- removed the U27 at (54.8, 155.8)
- removed the U27 at (320.2, -27.3)
- removed the U4 at (38.3, 155.8)
- removed the U4 at (204.9, 65.8)
- removed the U5 at (219.2, 57.1)
- removed the U5 at (161.9, 103.0)
- removed the U6 at (304.8, -22.6)
- removed the U6 at (136.2, 181.5)
- removed USB2: TYPE-C 16PIN 2MD(073), lcsc:USB-C-SMD_TYPE-C-6PIN-2MD-073
- removed Y2: 32.768KHz, lcsc:FC-135R_L3.2-W1.5
- added C217: 22uF, Capacitor_SMD:C_0603_1608Metric, F.Cu at (1237.5, 506.1)
- added C218: 22uF, Capacitor_SMD:C_0603_1608Metric, F.Cu at (1166.5, 503.4)
- added C219: 22uF, Capacitor_SMD:C_0603_1608Metric, F.Cu at (1258.0, 547.3)
- added C220: 22uF, Capacitor_SMD:C_0603_1608Metric, F.Cu at (1186.0, 546.9)
- added C221: 22uF, Capacitor_SMD:C_0603_1608Metric, F.Cu at (1218.0, 548.3)
- added C222: 22uF, Capacitor_SMD:C_0603_1608Metric, F.Cu at (1198.2, 505.3)
- added C223: 22uF, Capacitor_SMD:C_0603_1608Metric, F.Cu at (1239.3, 506.1)
- added C224: 22uF, Capacitor_SMD:C_0603_1608Metric, F.Cu at (1168.4, 503.4)
- added C225: 22uF, Capacitor_SMD:C_0603_1608Metric, F.Cu at (1254.1, 547.2)
- added C226: 22uF, Capacitor_SMD:C_0603_1608Metric, F.Cu at (1184.2, 546.9)
- added C227: 22uF, Capacitor_SMD:C_0603_1608Metric, F.Cu at (1216.2, 548.3)
- added C228: 22uF, Capacitor_SMD:C_0603_1608Metric, F.Cu at (1202.0, 505.3)
- added C229: 22uF, Capacitor_SMD:C_0603_1608Metric, F.Cu at (1235.6, 506.1)
- added C230: 22uF, Capacitor_SMD:C_0603_1608Metric, F.Cu at (1164.5, 503.4)
- added C231: 22uF, Capacitor_SMD:C_0603_1608Metric, F.Cu at (1256.1, 547.3)
- added C232: 22uF, Capacitor_SMD:C_0603_1608Metric, F.Cu at (1182.4, 546.9)
- added C233: 22uF, Capacitor_SMD:C_0603_1608Metric, F.Cu at (1221.7, 548.3)
- added C234: 22uF, Capacitor_SMD:C_0603_1608Metric, F.Cu at (1170.3, 503.4)
- added D33: 1N4148WS_C917117, lcsc:SOD-323_L1.8-W1.3-LS2.5-RD, F.Cu at (624.0, 465.1)
- added D34: 1N4148WS_C917117, lcsc:SOD-323_L1.8-W1.3-LS2.5-RD, F.Cu at (630.3, 495.1)
- added D35: 1N4148WS_C917117, lcsc:SOD-323_L1.8-W1.3-LS2.5-RD, F.Cu at (636.5, 525.1)
- added D36: 1N4148WS_C917117, lcsc:SOD-323_L1.8-W1.3-LS2.5-RD, F.Cu at (642.8, 555.1)
- added D37: 1N4148WS_C917117, lcsc:SOD-323_L1.8-W1.3-LS2.5-RD, F.Cu at (649.0, 465.1)
- added D38: 1N4148WS_C917117, lcsc:SOD-323_L1.8-W1.3-LS2.5-RD, F.Cu at (655.3, 495.1)
- added D39: 1N4148WS_C917117, lcsc:SOD-323_L1.8-W1.3-LS2.5-RD, F.Cu at (661.5, 525.1)
- added D40: 1N4148WS_C917117, lcsc:SOD-323_L1.8-W1.3-LS2.5-RD, F.Cu at (667.8, 555.1)
- added D41: 1N4148WS_C917117, lcsc:SOD-323_L1.8-W1.3-LS2.5-RD, F.Cu at (674.0, 465.1)
- added D42: 1N4148WS_C917117, lcsc:SOD-323_L1.8-W1.3-LS2.5-RD, F.Cu at (680.3, 495.1)
- added D43: 1N4148WS_C917117, lcsc:SOD-323_L1.8-W1.3-LS2.5-RD, F.Cu at (686.5, 525.1)
- added D44: 1N4148WS_C917117, lcsc:SOD-323_L1.8-W1.3-LS2.5-RD, F.Cu at (692.8, 555.1)
- added D45: 1N4148WS_C917117, lcsc:SOD-323_L1.8-W1.3-LS2.5-RD, F.Cu at (699.0, 465.1)
- added D46: 1N4148WS_C917117, lcsc:SOD-323_L1.8-W1.3-LS2.5-RD, F.Cu at (705.3, 495.1)
- added D47: 1N4148WS_C917117, lcsc:SOD-323_L1.8-W1.3-LS2.5-RD, F.Cu at (711.5, 525.1)
- added D48: 1N4148WS_C917117, lcsc:SOD-323_L1.8-W1.3-LS2.5-RD, F.Cu at (717.8, 555.1)
- added D49: LED, lcsc:LED0603-RD, F.Cu at (221.3, 375.8)
- added J7: Conn_01x02_Socket, lcsc:CONN-TH_2P-P5.00_WJ500V-5.08-2P, F.Cu at (734.7, 415.4)
- added L15: 6.8uH, lcsc:IND-SMD_L3.2-W2.5_L3225, F.Cu at (1178.0, 502.6)
- added L8: EXC14CE900U, lcsc:FILTER-SMD_4P-L0.9-W0.7-P0.50-BL, F.Cu at (1255.0, 461.6)
- added L9: 6.8uH, Inductor_SMD:L_6.3x6.3_H3, F.Cu at (1360.5, 585.1)
- added R128: 9.09K, Resistor_SMD:R_0402_1005Metric, F.Cu at (1194.6, 555.4)
- added R129: 100K, Resistor_SMD:R_0402_1005Metric, F.Cu at (1231.6, 558.8)
- added R130: 9.09K, Resistor_SMD:R_0402_1005Metric, F.Cu at (1230.1, 556.8)
- added R131: 100K, Resistor_SMD:R_0402_1005Metric, F.Cu at (1181.7, 513.9)
- added R132: 43.2K, Resistor_SMD:R_0402_1005Metric, F.Cu at (1180.3, 512.0)
- added R133: 10k, Resistor_SMD:R_0402_1005Metric, F.Cu at (405.2, 376.0)
- added R134: 4.7k, Resistor_SMD:R_0402_1005Metric, F.Cu at (405.2, 377.9)
- added R135: 10k, Resistor_SMD:R_0402_1005Metric, F.Cu at (405.2, 379.9)
- added U12: ~, lcsc:SW-TH_6P-L7.0-W7.0-P2.00_7-7-ZS, F.Cu at (260.5, 387.1)
- added U26: TPS54202DDC, Package_TO_SOT_SMD:SOT-23-6, F.Cu at (1208.4, 606.9)
- added U27: W29N02KVSIAF, lcsc:TSOP-48_L12.0-W18.4-P0.50-LS20.0-TL, F.Cu at (369.6, 450.7)
- added U38: LMR33630ADDAR, lcsc:ESOP-8_L4.9-W3.9-P1.27-LS6.0-TL-EP, F.Cu at (1227.9, 553.2)
- added U39: LMR33630ADDAR, lcsc:ESOP-8_L4.9-W3.9-P1.27-LS6.0-TL-EP, F.Cu at (1178.0, 508.5)
- added U4: NE5532DR, lcsc:SOIC-8_L4.9-W3.9-P1.27-LS6.0-BL, F.Cu at (642.9, 365.6)
- added U5: NE5532DR, lcsc:SOIC-8_L4.9-W3.9-P1.27-LS6.0-BL, F.Cu at (338.2, 337.3)
- added U6: NE5532DR, lcsc:SOIC-8_L4.9-W3.9-P1.27-LS6.0-BL, F.Cu at (460.9, 337.7)
- added USB1: TYPE-C 16PIN 2MD(073), lcsc:USB-C-SMD_TYPE-C-6PIN-2MD-073, F.Cu at (1255.0, 471.7)
- added Y1: 32.768KHz, lcsc:FC-135R_L3.2-W1.5, F.Cu at (400.4, 419.4)
- C1, C39: value 100nF -> 2.2uF
- C100, C145, C146, C155, C98, C99: value 0.1uF -> 100nF
- C101, C102, C103: value 100nF -> 220uF; footprint Capacitor_SMD:C_0402_1005Metric -> Capacitor_THT:CP_Radial_D8.0mm_P3.50mm
- C104: value 0.1uF -> 220uF; footprint Capacitor_SMD:C_0402_1005Metric -> Capacitor_THT:CP_Radial_D8.0mm_P3.50mm
- C105, C106, C107: value 1uF -> 680nF; footprint Capacitor_SMD:C_0402_1005Metric -> Capacitor_SMD:C_0603_1608Metric
- C108: value 1nF -> 680nF; footprint Capacitor_SMD:C_0402_1005Metric -> Capacitor_SMD:C_0603_1608Metric
- C109: value 1nF -> 1uF; footprint Capacitor_SMD:C_0402_1005Metric -> Capacitor_SMD:C_0603_1608Metric
- C11, C18, C80: value 2.2uF -> 0.1uF
- C110, C111, C112, C113: value 220nF -> 1uF; footprint Capacitor_SMD:C_0402_1005Metric -> Capacitor_SMD:C_0603_1608Metric
- C114, C115: value 100nF -> 1uF; footprint Capacitor_SMD:C_0402_1005Metric -> Capacitor_SMD:C_0603_1608Metric
- C116: value 220uF -> 1uF; footprint Capacitor_THT:CP_Radial_D8.0mm_P3.50mm -> Capacitor_SMD:C_0603_1608Metric
- C117: value 220uF -> 0.1uF; footprint Capacitor_THT:CP_Radial_D8.0mm_P3.50mm -> Capacitor_SMD:C_0603_1608Metric
- C118, C119: value 680nF -> 10nF; footprint Capacitor_SMD:C_0402_1005Metric -> Capacitor_SMD:C_0603_1608Metric
- C12, C3, C7: value 0.1uF -> 2.2uF
- C120, C121: value 1uF -> 10nF; footprint Capacitor_SMD:C_0402_1005Metric -> Capacitor_SMD:C_0603_1608Metric
- C122, C123, C176, C41: footprint Capacitor_SMD:C_0402_1005Metric -> Capacitor_SMD:C_0603_1608Metric
- C124, C127, C50, C61: value 1uF -> 0.1uF
- C125: value 680nF -> 2.2uF; footprint Capacitor_SMD:C_0402_1005Metric -> Capacitor_THT:CP_Radial_D8.0mm_P2.50mm
- C126: value 680nF -> 0.1uF
- C128: footprint Capacitor_SMD:C_0402_1005Metric -> Capacitor_THT:CP_Radial_D5.0mm_P2.00mm
- C129, C132: value 10nF -> 10uF
- C13, C14, C147, C15, C150, C152, C153, C16: value 10uF -> 0.1uF; footprint Capacitor_THT:CP_Radial_D8.0mm_P3.50mm -> Capacitor_SMD:C_0402_1005Metric
- C130: value 10nF -> 0.1uF
- C131: value 100nF -> 0.1uF; footprint Capacitor_SMD:C_0402_1005Metric -> Capacitor_THT:CP_Radial_D5.0mm_P2.00mm
- C136, C148: value 0.1uF -> 1uF; footprint Capacitor_SMD:C_0402_1005Metric -> Capacitor_THT:CP_Radial_D5.0mm_P2.00mm
- C137: value 220pF -> 10uF
- C138: value 220pF -> 0.1uF
- C140, C151: value 1uF -> 100nF; footprint Capacitor_THT:CP_Radial_D5.0mm_P2.00mm -> Capacitor_SMD:C_0402_1005Metric
- C141: footprint Capacitor_THT:CP_Radial_D5.0mm_P2.00mm -> Capacitor_SMD:C_0402_1005Metric
- C142: value 0.1uF -> 220pF
- C143, C167: value 0.1uF -> 10uF; footprint Capacitor_SMD:C_0402_1005Metric -> Capacitor_THT:CP_Radial_D8.0mm_P3.50mm
- C144: value 2.2uF -> 100nF; footprint Capacitor_THT:CP_Radial_D8.0mm_P2.50mm -> Capacitor_SMD:C_0402_1005Metric
- C149: value 1uF -> 220pF; footprint Capacitor_THT:CP_Radial_D5.0mm_P2.00mm -> Capacitor_SMD:C_0402_1005Metric
- C154: value 22pF -> 22uF
- C157: value 0.1uF -> 22uF
- C159: value 47pF -> 100nF
- C160, C162: value 22uF -> 10uF; footprint Capacitor_SMD:C_0603_1608Metric -> Capacitor_THT:CP_Radial_D8.0mm_P3.50mm
- C161, C172: value 22uF -> 100nF; footprint Capacitor_SMD:C_0603_1608Metric -> Capacitor_SMD:C_0402_1005Metric
- C163, C59, C60: value 22uF -> 0.1uF; footprint Capacitor_SMD:C_0603_1608Metric -> Capacitor_SMD:C_0402_1005Metric
- C164: value 10uF -> 100nF; footprint Capacitor_SMD:C_0603_1608Metric -> Capacitor_SMD:C_0402_1005Metric
- C165: value 220nF -> 1uF; footprint Capacitor_SMD:C_0603_1608Metric -> Capacitor_SMD:C_0402_1005Metric
- C166: value 1uF -> 100nF
- C168: value 47pF -> 5.1pF
- C169: value 22uF -> 5.1pF; footprint Capacitor_SMD:C_0603_1608Metric -> Capacitor_SMD:C_0402_1005Metric
- C17: value 10uF -> 2.2uF; footprint Capacitor_THT:CP_Radial_D8.0mm_P3.50mm -> Capacitor_SMD:C_0402_1005Metric
- C170, C171: value 22uF -> 5.6pF; footprint Capacitor_SMD:C_0603_1608Metric -> Capacitor_SMD:C_0402_1005Metric
- C173: value 22uF -> 22pF
- C174: value 22uF -> 100nF
- C175, C178: value 10uF -> 100nF
- C177, C179, C180, C181: value 0.1uF -> 10uF; footprint Capacitor_SMD:C_0402_1005Metric -> Capacitor_SMD:C_0603_1608Metric
- C182, C183: value 22uF -> 220nF; footprint Capacitor_SMD:C_0402_1005Metric -> Capacitor_SMD:C_0603_1608Metric
- C184: footprint Capacitor_THT:CP_Radial_D8.0mm_P3.50mm -> Capacitor_SMD:C_0603_1608Metric
- C185, C186, C94, C96: value 0.1uF -> 220nF
- C187, C89, C90, C91: value 10uF -> 220nF; footprint Capacitor_THT:CP_Radial_D8.0mm_P3.50mm -> Capacitor_SMD:C_0402_1005Metric
- C189, C194, C68, C82: value 0.1uF -> 1uF
- C19, C20: value 0.1uF -> 10uF; footprint Capacitor_SMD:C_0402_1005Metric -> lcsc:CAP-SMD_BD4.0-L4.3-W4.3-FD
- C190, C193: value 10uF -> 1uF; footprint Capacitor_THT:CP_Radial_D8.0mm_P3.50mm -> Capacitor_SMD:C_0402_1005Metric
- C191, C195: value 2.2uF -> 1uF
- C192: value 10uF -> 220nF; footprint Capacitor_THT:CP_Radial_D8.0mm_P3.50mm -> Capacitor_SMD:C_0603_1608Metric
- C197: value 100nF -> 1uF
- C198, C199, C200, C201, C202, C203: value 100nF -> 0.1uF
- C204, C205, C210: value 100nF -> 47pF
- C206: value 4.7uF -> 0.1uF
- C207: value 100nF -> 47pF; footprint Capacitor_SMD:C_0402_1005Metric -> Capacitor_SMD:C_0603_1608Metric
- C208, C209: value 2.2uF -> 47pF; footprint Capacitor_SMD:C_0402_1005Metric -> Capacitor_SMD:C_0603_1608Metric
- C21, C25: value 1nF -> 10uF; footprint Capacitor_SMD:C_0402_1005Metric -> lcsc:CAP-SMD_BD4.0-L4.3-W4.3-FD
- C211: value 100nF -> 22uF; footprint Capacitor_SMD:C_0402_1005Metric -> Capacitor_SMD:C_0603_1608Metric
- C212: value 100uF -> 22uF; footprint Capacitor_SMD:C_0402_1005Metric -> Capacitor_SMD:C_0603_1608Metric
- C213, C214: value 5.6pF -> 22uF; footprint Capacitor_SMD:C_0402_1005Metric -> Capacitor_SMD:C_0603_1608Metric
- C215, C216: value 5.1pF -> 22uF; footprint Capacitor_SMD:C_0402_1005Metric -> Capacitor_SMD:C_0603_1608Metric
- C22, C23, C24, C32, C33: value 1uF -> 10uF; footprint Capacitor_SMD:C_0402_1005Metric -> lcsc:CAP-SMD_BD4.0-L4.3-W4.3-FD
- C26: value 100nF -> 10uF; footprint Capacitor_SMD:C_0402_1005Metric -> lcsc:CAP-SMD_BD4.0-L4.3-W4.3-FD
- C27: value 220uF -> 10uF; footprint Capacitor_THT:CP_Radial_D8.0mm_P3.50mm -> lcsc:CAP-SMD_BD4.0-L4.3-W4.3-FD
- C28, C29, C30, C31: value 220nF -> 10uF; footprint Capacitor_SMD:C_0402_1005Metric -> lcsc:CAP-SMD_BD4.0-L4.3-W4.3-FD
- C34, C35: value 1uF -> 2.2uF
- C36, C37: value 10nF -> 2.2uF
- C38: value 1nF -> 2.2uF
- C40: value 220uF -> 0.1uF; footprint Capacitor_THT:CP_Radial_D8.0mm_P3.50mm -> Capacitor_SMD:C_0402_1005Metric
- C43: footprint Capacitor_SMD:C_0603_1608Metric -> Capacitor_SMD:C_0402_1005Metric
- C44, C63: value 10uF -> 0.1uF; footprint Capacitor_SMD:C_0603_1608Metric -> Capacitor_SMD:C_0402_1005Metric
- C45: value 220nF -> 0.1uF
- C46, C47: value 0.1uF -> 82nF; footprint Capacitor_SMD:C_0402_1005Metric -> PCM_Capacitor_THT_AKL:C_Rect_L4.0mm_W2.5mm_P2.50mm
- C48, C49: value 0.1uF -> 5.6nF; footprint Capacitor_SMD:C_0402_1005Metric -> PCM_Capacitor_THT_AKL:C_Rect_L4.0mm_W2.5mm_P2.50mm
- C56: value 47pF -> 82nF; footprint Capacitor_SMD:C_0402_1005Metric -> Capacitor_SMD:C_0603_1608Metric
- C57: value 22uF -> 82nF
- C58: value 22uF -> 100uF; footprint Capacitor_SMD:C_0603_1608Metric -> Capacitor_SMD:C_0402_1005Metric
- C62: value 220nF -> 0.1uF; footprint Capacitor_SMD:C_0603_1608Metric -> Capacitor_SMD:C_0402_1005Metric
- C64: value 10uF -> 5.6nF; footprint Capacitor_SMD:C_0603_1608Metric -> PCM_Capacitor_THT_AKL:C_Rect_L4.0mm_W2.5mm_P2.50mm
- C65: value 220nF -> 5.6nF; footprint Capacitor_SMD:C_0603_1608Metric -> PCM_Capacitor_THT_AKL:C_Rect_L4.0mm_W2.5mm_P2.50mm
- C69: value 47pF -> 1uF; footprint Capacitor_SMD:C_0603_1608Metric -> Capacitor_SMD:C_0402_1005Metric
- C70: value 22uF -> 1uF; footprint Capacitor_SMD:C_0603_1608Metric -> Capacitor_SMD:C_0402_1005Metric
- C71: value 22uF -> 1uF
- C72, C73: value 82nF -> 1uF; footprint Capacitor_SMD:C_0603_1608Metric -> Capacitor_SMD:C_0402_1005Metric
- C74: value 5.6nF -> 10nF; footprint PCM_Capacitor_THT_AKL:C_Rect_L4.0mm_W2.5mm_P2.50mm -> Capacitor_SMD:C_0402_1005Metric
- C75: value 82nF -> 0.1uF; footprint PCM_Capacitor_THT_AKL:C_Rect_L4.0mm_W2.5mm_P2.50mm -> Capacitor_SMD:C_0402_1005Metric
- C76, C79: value 5.6nF -> 0.1uF; footprint PCM_Capacitor_THT_AKL:C_Rect_L4.0mm_W2.5mm_P2.50mm -> Capacitor_SMD:C_0402_1005Metric
- C77: value 82nF -> 1nF; footprint PCM_Capacitor_THT_AKL:C_Rect_L4.0mm_W2.5mm_P2.50mm -> Capacitor_SMD:C_0402_1005Metric
- C78: value 5.6nF -> 100nF; footprint PCM_Capacitor_THT_AKL:C_Rect_L4.0mm_W2.5mm_P2.50mm -> Capacitor_SMD:C_0402_1005Metric
- C85: value 2.2uF -> 1nF
- C86: value 0.1uF -> 1nF
- C87, C88: value 10uF -> 1nF; footprint Capacitor_THT:CP_Radial_D8.0mm_P3.50mm -> Capacitor_SMD:C_0402_1005Metric
- C92, C93: value 2.2uF -> 220nF
- C95: value 1uF -> 220nF
- C97: value 2.2uF -> 100nF
- CN1: value USB-B-Female-90 -> DIN-504B-M10; footprint lcsc:USB-B_TH_USB-B-FEMALE-90 -> lcsc:CONN-TH_DIN-504B-M10
- D26: value 1N4148WT -> 1N4148WS_C917117; footprint Diode_SMD:D_SOD-523 -> lcsc:SOD-323_L1.8-W1.3-LS2.5-RD
- D27: value PESD15VL1BA -> 1N4148WS_C917117; footprint PCM_Diode_SMD_AKL:D_SOD-323_TVS -> lcsc:SOD-323_L1.8-W1.3-LS2.5-RD
- D28: value BAT54 -> 1N4148WS_C917117; footprint PCM_Package_TO_SOT_SMD_AKL:SOT-23 -> lcsc:SOD-323_L1.8-W1.3-LS2.5-RD
- D29, D30, D31: value LED -> 1N4148WS_C917117; footprint LED_SMD:LED_0603_1608Metric -> lcsc:SOD-323_L1.8-W1.3-LS2.5-RD
- D32: value SB520 -> 1N4148WS_C917117; footprint PCM_Diode_THT_AKL:D_DO-201AD_P12.70mm_Horizontal -> lcsc:SOD-323_L1.8-W1.3-LS2.5-RD
- D50: value 1N4148WS_C917117 -> 1N4148WT; footprint lcsc:SOD-323_L1.8-W1.3-LS2.5-RD -> Diode_SMD:D_SOD-523
- D51: value 1N4148WS_C917117 -> PESD15VL1BA; footprint lcsc:SOD-323_L1.8-W1.3-LS2.5-RD -> PCM_Diode_SMD_AKL:D_SOD-323_TVS
- D52, D53, D54: value 1N4148WS_C917117 -> LED; footprint lcsc:SOD-323_L1.8-W1.3-LS2.5-RD -> LED_SMD:LED_0603_1608Metric
- D55: value 1N4148WS_C917117 -> BAT54; footprint lcsc:SOD-323_L1.8-W1.3-LS2.5-RD -> PCM_Package_TO_SOT_SMD_AKL:SOT-23
- J1: value Conn_01x13_Pin -> PJ-625G; footprint Connector_PinHeader_2.54mm:PinHeader_1x13_P2.54mm_Vertical -> lcsc:AUDIO-TH_PJ-625G
- J10: value Conn_01x02_Socket -> Conn_01x08_Pin; footprint lcsc:CONN-TH_2P-P5.00_WJ500V-5.08-2P -> lcsc:CONN-TH_B8PS-VH-LF-SN
- J11: value Conn_01x08_Pin -> Conn_01x02_Socket; footprint lcsc:CONN-TH_B8PS-VH-LF-SN -> lcsc:CONN-TH_2P-P5.00_WJ500V-5.08-2P
- J2: value Conn_01x03_Pin -> PJ-625G; footprint Connector_PinHeader_2.54mm:PinHeader_1x03_P2.54mm_Vertical -> lcsc:AUDIO-TH_PJ-625G
- J3: value PJ-625G -> Conn_01x13_Pin; footprint lcsc:AUDIO-TH_PJ-625G -> Connector_PinHeader_2.54mm:PinHeader_1x13_P2.54mm_Vertical
- J4: value PJ-625G -> Conn_01x03_Pin; footprint lcsc:AUDIO-TH_PJ-625G -> Connector_PinHeader_2.54mm:PinHeader_1x03_P2.54mm_Vertical
- L10: value 10uH -> 8uH; footprint lcsc:IND-SMD_L11.0-W10.5_SL1050-330M -> lcsc:L1206
- L11: value 10uH -> 6.8uH; footprint lcsc:IND-SMD_L11.0-W10.5_SL1050-330M -> lcsc:IND-SMD_L3.2-W2.5_L3225
- L12: value 6.8uH -> 15uH; footprint Inductor_SMD:L_6.3x6.3_H3 -> lcsc:IND-SMD_L12.3-W12.3
- L13: value 6.8uH -> 15uH; footprint lcsc:IND-SMD_L3.2-W2.5_L3225 -> lcsc:IND-SMD_L12.3-W12.3
- L4: value 8uH -> 10uH; footprint lcsc:L1206 -> lcsc:IND-SMD_L11.0-W10.5_SL1050-330M
- L5: value 15uH -> 10uH; footprint lcsc:IND-SMD_L12.3-W12.3 -> lcsc:IND-SMD_L11.0-W10.5_SL1050-330M
- L6: value 27uH -> 10uH; footprint lcsc:IND-SMD_L4.8-W3.4 -> lcsc:IND-SMD_L11.0-W10.5_SL1050-330M
- L7: value 10uH -> 27uH; footprint lcsc:IND-SMD_L11.0-W10.5_SL1050-330M -> lcsc:IND-SMD_L4.8-W3.4
- R1, R2: value 1.5K -> 470K
- R10: value 100k -> 6K
- R100, R101, R99: value 10K -> 22
- R102, R98: value 100K -> 22
- R103: value NTCG163JF103FT1S -> 22; footprint lcsc:R0603 -> Resistor_SMD:R_0402_1005Metric
- R104: value 9.31K -> 1.5K
- R105: value 430K -> 0.01
- R106: value 22 -> 49.9
- R107: value 22 -> 50k
- R108: value 22 -> 2.61k
- R109: value 22 -> 10k
- R11: value 75k -> 6K
- R110: value 22 -> 100K
- R111: value 10K -> 500K
- R112, R127: value 10K -> 100K
- R113, R114: value 10K -> 0
- R117: value 0 -> 1K
- R12: value 47k -> 10K
- R121: value 10k -> 100K
- R122: value 1k -> 24.9K
- R123: value 220 -> 100K
- R124: value 33 -> 43.2K
- R125: value 10 -> 100K
- R126: value 10k -> 9.09K
- R13, R17: value 100k -> 10K
- R14, R15, R25: value 3.3 -> 10K
- R16: value 75k -> 10K
- R18: value 100k -> 5K
- R19, R20, R24: value 3.3 -> 6K
- R23: value 10k -> 10K
- R26: value 100k -> 33
- R27: value 10K -> 220
- R28, R84: value 10K -> 10
- R31, R37, R38, R95: value 100K -> 1K
- R32: value 24.9K -> 1K
- R33, R34: value 100K -> 10K
- R35: value 100K -> 470
- R36: value 43.2K -> 1K
- R39: value 9.09K -> 1K
- R40: value 100K -> 47k
- R41: value 100K -> 75k
- R42: value 9.09K -> 47k
- R43: value 49.9 -> 75k
- R44: value 50k -> 100k
- R45: value 2.61k -> 100k
- R46, R49: value 470K -> 100k
- R47, R48: value 470K -> 6K
- R5, R6: value 6K -> 470K
- R50: value 10K -> 100k
- R51: value 10K -> 10k
- R53: value 10K -> 6K
- R54: value 1k -> 1K
- R55, R56, R57: value 22 -> 6K
- R58: value 200K -> 10K
- R59, R60, R61, R62, R63: value 6K -> 10K
- R64, R65, R67, R68: value 6K -> 3.3
- R66, R69: value 100K -> 3.3
- R73: value 6K -> 2
- R75: value 6K -> 100K
- R76: value 1K -> 32.4K
- R78, R80, R89: value 1K -> 100K
- R79, R94: value 1K -> 10K
- R81: value 1K -> 22.1K
- R82: value 10K -> 0.01
- R83, R87: value 10K -> 1k
- R85: value 10K -> 200K
- R86: value 22.1K -> 1.5K
- R88: value 32.4K -> 9.31K
- R9: value 47k -> 6K
- R90: value 100K -> NTCG163JF103FT1S; footprint Resistor_SMD:R_0402_1005Metric -> lcsc:R0603
- R91: value 10 -> 430K
- R92: value 2 -> 10K
- R93: value 0.01 -> 10K
- R96: value 0.01 -> 22
- R97: value 500K -> 22
- SW10, SW19, SW20, SW33, SW34, SW5: value TS-1003ST-26 -> RotaryEncoder; footprint lcsc:SW-SMD_4P-L12.0-W12.0-P5.00-LS15.4 -> lcsc:SW-TH_EC12EXXXX
- SW49: value RotaryEncoder_Switch -> TS-1003ST-26; footprint lcsc:SW-TH_EC11E1820402 -> lcsc:SW-SMD_4P-L12.0-W12.0-P5.00-LS15.4
- SW50, SW51, SW52, SW53, SW54, SW55: value RotaryEncoder -> TS-1003ST-26; footprint lcsc:SW-TH_EC12EXXXX -> lcsc:SW-SMD_4P-L12.0-W12.0-P5.00-LS15.4
- SW58: value TS-1003ST-26 -> SW_Push; footprint lcsc:SW-SMD_4P-L12.0-W12.0-P5.00-LS15.4 -> Button_Switch_SMD:SW_SPST_CK_RS282G05A3
- SW59: value SW_Push -> RotaryEncoder_Switch; footprint Button_Switch_SMD:SW_SPST_CK_RS282G05A3 -> lcsc:SW-TH_EC11E1820402
- U1: value NE5532DR -> PCM5122PW; footprint lcsc:SOIC-8_L4.9-W3.9-P1.27-LS6.0-BL -> Package_SO:TSSOP-28_4.4x9.7mm_P0.65mm
- U11, U7, U8: value ~ -> NE5532DR; footprint lcsc:SW-TH_6P-L7.0-W7.0-P2.00_7-7-ZS -> lcsc:SOIC-8_L4.9-W3.9-P1.27-LS6.0-BL
- U13, U14: value LMR33630ADDAR -> ~; footprint lcsc:ESOP-8_L4.9-W3.9-P1.27-LS6.0-TL-EP -> lcsc:SW-TH_6P-L7.0-W7.0-P2.00_7-7-ZS
- U15: value TPS54202DDC -> TS5A23159RSER; footprint Package_TO_SOT_SMD:SOT-23-6 -> lcsc:UQFN-10_L2.0-W1.5-P0.50-BL-EP
- U16: value PCM5122PW -> NE5532DR; footprint Package_SO:TSSOP-28_4.4x9.7mm_P0.65mm -> lcsc:SOIC-8_L4.9-W3.9-P1.27-LS6.0-BL
- U17: value USBLC6-2P6 -> TPA6120A2DWP; footprint Package_TO_SOT_SMD:SOT-666 -> lcsc:HSOP-20_L12.8-W7.5-P1.27-LS10.3-BL-EP3.3
- U18, U19: value NE5532DR -> TPA3116D2DAD_C2865736; footprint lcsc:SOIC-8_L4.9-W3.9-P1.27-LS6.0-BL -> lcsc:HTSSOP-32_L11.0-W6.1-P0.65-LS8.1-BL
- U2: value TPA3116D2DAD_C2865736 -> PCM5122PW; footprint lcsc:HTSSOP-32_L11.0-W6.1-P0.65-LS8.1-BL -> Package_SO:TSSOP-28_4.4x9.7mm_P0.65mm
- U21: value TPA6120A2DWP -> CY8CMBR3116-LQXIT; footprint lcsc:HSOP-20_L12.8-W7.5-P1.27-LS10.3-BL-EP3.3 -> lcsc:QFN-24_L4.0-W4.0-P0.50-BL-EP2.6
- U22, U24: value NE5532DR -> FPC-05F-6PH20; footprint lcsc:SOIC-8_L4.9-W3.9-P1.27-LS6.0-BL -> lcsc:FPC-SMD_6P-P0.50_XUNPU_FPC-05F-6PH20
- U23: value TS5A23159RSER -> NE5532DR; footprint lcsc:UQFN-10_L2.0-W1.5-P0.50-BL-EP -> lcsc:SOIC-8_L4.9-W3.9-P1.27-LS6.0-BL
- U25: value NE5532DR -> BQ24610; footprint lcsc:SOIC-8_L4.9-W3.9-P1.27-LS6.0-BL -> Package_DFN_QFN:VQFN-24-1EP_4x4mm_P0.5mm_EP2.45x2.45mm
- U28: value NE5532DR -> USBLC6-2P6; footprint lcsc:SOIC-8_L4.9-W3.9-P1.27-LS6.0-BL -> Package_TO_SOT_SMD:SOT-666
- U29: value NE5532DR -> TUSB422IYFPR; footprint lcsc:SOIC-8_L4.9-W3.9-P1.27-LS6.0-BL -> lcsc:DSBGA-9_L1.4-W1.3-R3-C3-P0.40-BL
- U3: value CY8CMBR3116-LQXIT -> PCM5122PW; footprint lcsc:QFN-24_L4.0-W4.0-P0.50-BL-EP2.6 -> Package_SO:TSSOP-28_4.4x9.7mm_P0.65mm
- U30: value TPA3116D2DAD_C2865736 -> SIS412DN-T1-GE3-ES; footprint lcsc:HTSSOP-32_L11.0-W6.1-P0.65-LS8.1-BL -> lcsc:PDFN-8_L3.1-W3.1-P0.65-LS3.4-BL
- U31: value BQ24610 -> SIS412DN-T1-GE3-ES; footprint Package_DFN_QFN:VQFN-24-1EP_4x4mm_P0.5mm_EP2.45x2.45mm -> lcsc:PDFN-8_L3.1-W3.1-P0.65-LS3.4-BL
- U32: value TUSB422IYFPR -> ~; footprint lcsc:DSBGA-9_L1.4-W1.3-R3-C3-P0.40-BL -> lcsc:CRYSTAL-SMD_4P-L3.2-W2.5-BL_SIT8008BI
- U33: value SIS412DN-T1-GE3-ES -> HS20HS072RX; footprint lcsc:PDFN-8_L3.1-W3.1-P0.65-LS3.4-BL -> lcsc:OLED-SMD_HS20HS072RX
- U34: value SIS412DN-T1-GE3-ES -> LMR33630ADDAR; footprint lcsc:PDFN-8_L3.1-W3.1-P0.65-LS3.4-BL -> lcsc:ESOP-8_L4.9-W3.9-P1.27-LS6.0-TL-EP
- U36: value FPC-05F-6PH20 -> LMR33630ADDAR; footprint lcsc:FPC-SMD_6P-P0.50_XUNPU_FPC-05F-6PH20 -> lcsc:ESOP-8_L4.9-W3.9-P1.27-LS6.0-TL-EP
- U37: value ~ -> LMR33630ADDAR; footprint lcsc:CRYSTAL-SMD_4P-L3.2-W2.5-BL_SIT8008BI -> lcsc:ESOP-8_L4.9-W3.9-P1.27-LS6.0-TL-EP
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Connections:
- AUDIO1 pad 4: Main On/Off Switch -> GND
- C1 pad 1: VBUS -> Net-(U1-CAPP)
- C1 pad 2: Main On/Off Switch -> Net-(U1-CAPM)
- C10 pad 1: Main On/Off Switch -> +3.3V
- C10 pad 2: Net-(U4-LDOO) -> GND
- C100 pad 1: Main On/Off Switch -> GND
- C100 pad 2: RX MIDI -> +12V
- C101 pad 1: +3.3VA -> +12V
- C101 pad 2: Main On/Off Switch -> GND
- C102 pad 1: RX MIDI -> +12V
- C102 pad 2: Main On/Off Switch -> GND
- C103 pad 1: RX MIDI -> +12V
- C103 pad 2: Main On/Off Switch -> GND
- C104 pad 1: Main On/Off Switch -> +12V
- C104 pad 2: +12V -> GND
- C105 pad 1: Net-(U30-RINP) -> GND
- C105 pad 2: TWEET SUM BUFF -> TWEET AMP P
- C106 pad 1: Net-(U30-RINN) -> TWEET AMP N
- C106 pad 2: TWEET SUM BUFF N -> GND
- C107 pad 1: Net-(U30-LINP) -> GND
- C107 pad 2: WOOF SUM BUFF -> WOOF AMP P
- C108 pad 1: Main On/Off Switch -> WOOF AMP N
- C108 pad 2: +12V -> GND
- C109 pad 1: Main On/Off Switch -> GND
- C109 pad 2: +12V -> SUB AMP P
- C11 pad 1: Main On/Off Switch -> GND
- C11 pad 2: Net-(U4-VNEG) -> Net-(U2-LDOO)
- C110 pad 1: Net-(U30-OUTPR) -> SUB AMP N
- C110 pad 2: Net-(U30-BSPR) -> GND
- C111 pad 1: Net-(U30-OUTNR) -> GND
- C111 pad 2: Net-(U30-BSNR) -> TWEET AMP P
- C112 pad 1: Net-(U30-OUTPL) -> TWEET AMP N
- C112 pad 2: Net-(U30-BSPL) -> GND
- C113 pad 1: Net-(U30-BSNL) -> GND
- C113 pad 2: Net-(U30-OUTNL) -> WOOF AMP P
- C114 pad 1: Main On/Off Switch -> WOOF AMP N
- C114 pad 2: +12V -> GND
- C115 pad 1: Main On/Off Switch -> GND
- C115 pad 2: +12V -> SUB AMP P
- C116 pad 1: +12V -> SUB AMP N
- C116 pad 2: Main On/Off Switch -> GND
- C117 pad 1: +12V -> GND
- C117 pad 2: Main On/Off Switch -> -12V
- C118 pad 1: Main On/Off Switch -> GND
- C118 pad 2: TWEET AMP P -> Net-(C118-Pad2)
- C119 pad 1: TWEET AMP N -> Net-(C119-Pad1)
- C119 pad 2: Main On/Off Switch -> GND
- C12 pad 1: +3.3VA -> GND
- C12 pad 2: Main On/Off Switch -> Net-(U2-VNEG)
- C120 pad 1: Main On/Off Switch -> GND
- C120 pad 2: TWEET AMP P -> Net-(C120-Pad2)
- C121 pad 1: TWEET AMP N -> Net-(C121-Pad1)
- C121 pad 2: Main On/Off Switch -> GND
- C122 pad 1: Main On/Off Switch -> GND
- C123 pad 2: Main On/Off Switch -> GND
- C124 pad 1: Net-(U30-LINN) -> GND
- C124 pad 2: WOOF SUM BUFF N -> +12V
- C125 pad 1: Main On/Off Switch -> Net-(C125-Pad1)
- C125 pad 2: WOOF AMP P -> GND
- C126 pad 1: WOOF AMP N -> Net-(Q2-D)
- C126 pad 2: Main On/Off Switch -> Net-(Q1-G)
- C127 pad 1: Main On/Off Switch -> GND
- C127 pad 2: WOOF AMP P -> Net-(U25-ACP)
- C128 pad 1: WOOF AMP N -> Net-(U25-CE)
- C128 pad 2: Main On/Off Switch -> GND
- C129 pad 1: Main On/Off Switch -> +12V
- C129 pad 2: Net-(C129-Pad2) -> GND
- C13 pad 2: Main On/Off Switch -> GND
- C130 pad 1: Net-(C130-Pad1) -> Net-(U25-ACP)
- C130 pad 2: Main On/Off Switch -> SYS
- C131 pad 1: Main On/Off Switch -> Net-(U25-TTC)
- C131 pad 2: Net-(C131-Pad2) -> GND
- C132 pad 2: Main On/Off Switch -> GND
- C133 pad 1: Main On/Off Switch -> +12V
- C133 pad 2: -12V -> GND
- C134 pad 1: +12V -> GND
- C134 pad 2: Main On/Off Switch -> +3.3V
- C136 pad 1: Main On/Off Switch -> Net-(U25-VCC)
- C136 pad 2: -12V -> GND
- C137 pad 1: Net-(U32-CC2) -> +12V
- C137 pad 2: Main On/Off Switch -> -12V
- C138 pad 1: Net-(U32-CC1) -> Net-(U25-TS)
- C138 pad 2: Main On/Off Switch -> GND
- C139 pad 1: RX MIDI -> +12V
- C139 pad 2: Main On/Off Switch -> -12V
- C14 pad 1: Net-(U4-VCOM/DEMP) -> +3.3VA
- C14 pad 2: Main On/Off Switch -> GND
- C140 pad 1: Net-(U31-CE) -> +3.3V
- C140 pad 2: Main On/Off Switch -> GND
- C141 pad 1: Net-(U31-TTC) -> +3.3V
- C141 pad 2: Main On/Off Switch -> GND
- C142 pad 1: Net-(Q2-D) -> Net-(U29-CC2)
- C142 pad 2: Net-(Q1-G) -> GND
- C143 pad 1: Net-(D28-K) -> SYS
- C143 pad 2: Net-(U31-PH) -> GND
- C144 pad 1: Net-(C144-Pad1) -> +3.3V
- C144 pad 2: Main On/Off Switch -> GND
- C145 pad 1: Net-(U31-ACP) -> VBUS
- C145 pad 2: SYS -> GND
- C146 pad 1: Main On/Off Switch -> +3.3V
- C146 pad 2: Net-(U31-ACP) -> GND
- C147 pad 1: SYS -> Net-(U26-SW)
- C147 pad 2: Main On/Off Switch -> Net-(U26-BOOT)
- C148 pad 1: Net-(Q3-G) -> Net-(D55-A)
- C148 pad 2: SYS -> GND
- C149 pad 1: Net-(D28-A) -> Net-(U29-CC1)
- C149 pad 2: Main On/Off Switch -> GND
- C15 pad 1: RX MIDI -> +3.3V
- C15 pad 2: Main On/Off Switch -> GND
- C150 pad 1: SYS -> GND
- C150 pad 2: Main On/Off Switch -> +3.3V
- C151 pad 1: Net-(U31-VCC) -> +3.3V
- C151 pad 2: Main On/Off Switch -> GND
- C152 pad 1: +BATT -> Net-(D55-K)
- C152 pad 2: Main On/Off Switch -> Net-(U25-PH)
- C153 pad 1: +BATT -> GND
- C153 pad 2: Main On/Off Switch -> -12V
- C154 pad 1: Net-(U31-VFB) -> GND
- C154 pad 2: +BATT -> -12V
- C155 pad 1: +BATT -> +3.3V
- C155 pad 2: Net-(U31-SRP) -> GND
- C156 pad 1: Net-(U31-SRP) -> Net-(U25-SRP)
- C156 pad 2: Main On/Off Switch -> GND
- C157 pad 1: Net-(U31-TS) -> GND
- C157 pad 2: Main On/Off Switch -> -12V
- C158 pad 1: Net-(U13-SW) -> +BATT
- C158 pad 2: Net-(U13-BOOT) -> Net-(U25-SRP)
- C159 pad 1: RX MIDI -> +3.3V
- C159 pad 2: Net-(U13-FB) -> GND
- C16 pad 1: Net-(U4-LDOO) -> GND
- C16 pad 2: Main On/Off Switch -> Net-(U3-LDOO)
- C160 pad 1: RX MIDI -> +BATT
- C160 pad 2: Main On/Off Switch -> GND
- C161 pad 1: RX MIDI -> +3.3V
- C161 pad 2: Main On/Off Switch -> GND
- C162 pad 1: RX MIDI -> +BATT
- C162 pad 2: Main On/Off Switch -> GND
- C163 pad 1: RX MIDI -> Net-(Q3-G)
- C163 pad 2: Main On/Off Switch -> SYS
- C164 pad 1: SYS -> +3.3V
- C164 pad 2: Main On/Off Switch -> GND
- C165 pad 1: SYS -> +3.3V
- C165 pad 2: Main On/Off Switch -> GND
- C166 pad 1: Net-(U14-VCC) -> +3.3V
- C166 pad 2: Main On/Off Switch -> GND
- C167 pad 1: Net-(U14-SW) -> SYS
- C167 pad 2: Net-(U14-BOOT) -> GND
- C168 pad 1: +12V -> GND
- C168 pad 2: Net-(U14-FB) -> Net-(VQ1-PC14-OSC32_IN)
- C169 pad 1: +12V -> GND
- C169 pad 2: Main On/Off Switch -> Net-(VQ1-PC15-OSC32_OUT)
- C17 pad 1: +3.3VA -> GND
- C17 pad 2: Main On/Off Switch -> Net-(U3-VNEG)
- C170 pad 1: +12V -> GND
- C170 pad 2: Main On/Off Switch -> Net-(VQ1-PH0-OSC_IN)
- C171 pad 1: +12V -> GND
- C171 pad 2: Main On/Off Switch -> Net-(VQ1-PH1-OSC_OUT)
- C172 pad 1: +12V -> +3.3VA
- C172 pad 2: Main On/Off Switch -> GND
- C173 pad 1: +12V -> Net-(U25-VFB)
- C173 pad 2: Main On/Off Switch -> +BATT
- C174 pad 1: +12V -> +3.3V
- C174 pad 2: Main On/Off Switch -> GND
- C175 pad 1: +12V -> +3.3V
- C175 pad 2: Main On/Off Switch -> GND
- C176 pad 1: +12V -> VBUS
- C176 pad 2: Main On/Off Switch -> GND
- C177 pad 1: +12V -> SYS
- C177 pad 2: Main On/Off Switch -> GND
- C178 pad 1: +12V -> +3.3V
- C178 pad 2: -12V -> GND
- C179 pad 1: +12V -> SYS
- C179 pad 2: -12V -> GND
- C18 pad 1: HEADPHONE DAC L -> +3.3VA
- C18 pad 2: Main On/Off Switch -> GND
- C180 pad 1: Net-(U15-SW) -> SYS
- C180 pad 2: Net-(U15-BOOT) -> GND
- C181 pad 1: Main On/Off Switch -> SYS
- C181 pad 2: -12V -> GND
- C182 pad 1: Main On/Off Switch -> VBUS
- C182 pad 2: -12V -> GND
- C183 pad 1: Main On/Off Switch -> SYS
- C183 pad 2: -12V -> GND
- C184 pad 1: RX MIDI -> +BATT
- C184 pad 2: Main On/Off Switch -> GND
- C185 pad 1: RX MIDI -> SYS
- C185 pad 2: Main On/Off Switch -> GND
- C186 pad 1: Main On/Off Switch -> SYS
- C186 pad 2: Net-(U16-LDOO) -> GND
- C187 pad 1: Net-(U16-LDOO) -> SYS
- C187 pad 2: Main On/Off Switch -> GND
- C188 pad 1: Main On/Off Switch -> Net-(C188-Pad1)
- C188 pad 2: Net-(U16-VNEG) -> GND
- C189 pad 1: +3.3VA -> Net-(U34-VCC)
- C189 pad 2: Main On/Off Switch -> GND
- C19 pad 1: Main On/Off Switch -> +3.3VA
- C19 pad 2: -12V -> GND
- C190 pad 1: +3.3VA -> Net-(U35-VCC)
- C190 pad 2: Main On/Off Switch -> GND
- C191 pad 1: Net-(U16-CAPP) -> GND
- C191 pad 2: Net-(U16-CAPM) -> 3.3BATT
- C192 pad 1: Net-(U16-VCOM/DEMP) -> +BATT
- C192 pad 2: Main On/Off Switch -> GND
- C193 pad 1: +3.3VA -> Net-(U36-VCC)
- C193 pad 2: Main On/Off Switch -> GND
- C194 pad 1: +3.3VA -> Net-(U37-VCC)
- C194 pad 2: Main On/Off Switch -> GND
- C195 pad 1: SPEAKER DAC R -> Net-(U38-VCC)
- C195 pad 2: Main On/Off Switch -> GND
- C196 pad 1: SPEAKER DAC L -> Net-(C188-Pad1)
- C196 pad 2: Main On/Off Switch -> GND
- C197 pad 1: RX MIDI -> Net-(U39-VCC)
- C197 pad 2: Main On/Off Switch -> GND
- C198 pad 1: RX MIDI -> GND
- C198 pad 2: Main On/Off Switch -> +3.3V
- C199 pad 1: RX MIDI -> Net-(U34-SW)
- C199 pad 2: Main On/Off Switch -> Net-(U34-BOOT)
- C2 pad 1: Net-(U4-CAPP) -> Net-(U2-CAPP)
- C2 pad 2: Net-(U4-CAPM) -> Net-(U2-CAPM)
- C20 pad 1: Main On/Off Switch -> Net-(U1-VCOM/DEMP)
- C20 pad 2: +12V -> GND
- C200 pad 1: RX MIDI -> Net-(U35-SW)
- C200 pad 2: Main On/Off Switch -> Net-(U35-BOOT)
- C201 pad 1: RX MIDI -> Net-(U36-SW)
- C201 pad 2: Main On/Off Switch -> Net-(U36-BOOT)
- C202 pad 1: RX MIDI -> Net-(U37-SW)
- C202 pad 2: Main On/Off Switch -> Net-(U37-BOOT)
- C203 pad 1: RX MIDI -> Net-(U38-SW)
- C203 pad 2: Main On/Off Switch -> Net-(U38-BOOT)
- C204 pad 1: RX MIDI -> +5V
- C204 pad 2: Main On/Off Switch -> Net-(U34-FB)
- C205 pad 1: RX MIDI -> +3.3V
- C205 pad 2: Main On/Off Switch -> Net-(U35-FB)
- C206 pad 1: RX MIDI -> Net-(U39-SW)
- C206 pad 2: Main On/Off Switch -> Net-(U39-BOOT)
- C207 pad 1: RX MIDI -> +12V
- C207 pad 2: Main On/Off Switch -> Net-(U36-FB)
- C208 pad 1: Net-(C208-Pad1) -> +12V
- C208 pad 2: Main On/Off Switch -> Net-(U37-FB)
- C209 pad 1: Net-(C208-Pad1) -> +12V
- C209 pad 2: Main On/Off Switch -> Net-(U38-FB)
- C21 pad 1: Net-(U2-SYNC) -> +3.3V
- C21 pad 2: Main On/Off Switch -> GND
- C210 pad 1: RX MIDI -> 3.3BATT
- C210 pad 2: Main On/Off Switch -> Net-(U39-FB)
- C211 pad 1: RX MIDI -> +5V
- C211 pad 2: Main On/Off Switch -> GND
- C212 pad 1: RX MIDI -> +3.3V
- C212 pad 2: Main On/Off Switch -> GND
- C213 pad 1: Main On/Off Switch -> +12V
- C213 pad 2: Net-(VQ1-PH1-OSC_OUT) -> GND
- C214 pad 1: Main On/Off Switch -> +12V
- C214 pad 2: Net-(VQ1-PH0-OSC_IN) -> GND
- C215 pad 1: Main On/Off Switch -> +12V
- C215 pad 2: Net-(VQ1-PC14-OSC32_IN) -> GND
- C216 pad 1: Main On/Off Switch -> +5V
- C216 pad 2: Net-(VQ1-PC15-OSC32_OUT) -> GND
- C22 pad 1: Net-(U2-GVDD) -> Net-(U1-LDOO)
- C22 pad 2: Main On/Off Switch -> GND
- C23 pad 1: Net-(U2-RINN) -> +3.3VA
- C23 pad 2: SUB SUM BUFF N -> GND
- C24 pad 1: Net-(U2-RINP) -> +3.3VA
- C24 pad 2: SUB SUM BUFF -> GND
- C25 pad 1: Main On/Off Switch -> Net-(U2-VCOM/DEMP)
- C25 pad 2: +12V -> GND
- C26 pad 1: Main On/Off Switch -> +3.3V
- C26 pad 2: +12V -> GND
- C27 pad 1: +12V -> Net-(U2-LDOO)
- C27 pad 2: Main On/Off Switch -> GND
- C28 pad 1: Net-(U2-OUTNR) -> +3.3VA
- C28 pad 2: Net-(U2-BSPR) -> GND
- C29 pad 1: Net-(U2-OUTNR) -> +3.3VA
- C29 pad 2: Net-(U2-BSNR) -> GND
- C3 pad 1: +3.3VA -> Net-(U3-CAPP)
- C3 pad 2: Main On/Off Switch -> Net-(U3-CAPM)
- C30 pad 1: Net-(U2-BSNL) -> Net-(U3-VCOM/DEMP)
- C30 pad 2: Net-(U2-OUTNL) -> GND
- C31 pad 1: Net-(U2-OUTNL) -> +3.3V
- C31 pad 2: Net-(U2-BSPL) -> GND
- C32 pad 1: SUB AMP N -> Net-(U3-LDOO)
- C32 pad 2: Main On/Off Switch -> GND
- C33 pad 1: Main On/Off Switch -> +3.3VA
- C33 pad 2: SUB AMP P -> GND
- C34 pad 1: Main On/Off Switch -> HEADPHONE DAC L
- C34 pad 2: SUB AMP P -> GND
- C35 pad 1: SUB AMP N -> HEADPHONE DAC R
- C35 pad 2: Main On/Off Switch -> GND
- C36 pad 1: Main On/Off Switch -> SPEAKER DAC L
- C36 pad 2: Net-(C36-Pad2) -> GND
- C37 pad 1: Net-(C37-Pad1) -> SPEAKER DAC R
- C37 pad 2: Main On/Off Switch -> GND
- C38 pad 1: Main On/Off Switch -> STEREO OUT DAC L
- C38 pad 2: +12V -> GND
- C39 pad 1: Main On/Off Switch -> STEREO OUT DAC R
- C39 pad 2: +12V -> GND
- C4 pad 1: Main On/Off Switch -> +3.3VA
- C4 pad 2: -12V -> GND
- C40 pad 1: +12V -> GND
- C40 pad 2: Main On/Off Switch -> -12V
- C41 pad 1: Main On/Off Switch -> GND
- C41 pad 2: -12V -> +12V
- C42 pad 1: Main On/Off Switch -> GND
- C42 pad 2: +12V -> -12V
- C43 pad 1: Main On/Off Switch -> GND
- C43 pad 2: +12V -> -12V
- C44 pad 1: SYS -> GND
- C44 pad 2: Main On/Off Switch -> +12V
- C45 pad 1: SYS -> GND
- C45 pad 2: Main On/Off Switch -> +12V
- C46 pad 1: Main On/Off Switch -> SPEAKER SUM BUFF
- C46 pad 2: -12V -> Net-(C46-Pad2)
- C47 pad 1: Main On/Off Switch -> Net-(C46-Pad2)
- C47 pad 2: +12V -> Net-(U7-IN1+)
- C48 pad 1: Main On/Off Switch -> GND
- C48 pad 2: -12V -> Net-(U7-IN2+)
- C49 pad 1: RX MIDI -> GND
- C49 pad 2: Main On/Off Switch -> Net-(U7-IN2+)
- C5 pad 1: Main On/Off Switch -> +3.3V
- C5 pad 2: +12V -> GND
- C50 pad 1: Net-(U30-GVDD) -> GND
- C50 pad 2: Main On/Off Switch -> -12V
- C51 pad 1: Main On/Off Switch -> GND
- C52 pad 1: Main On/Off Switch -> GND
- C53 pad 1: Main On/Off Switch -> GND
- C54 pad 1: Main On/Off Switch -> GND
- C55 pad 1: Net-(U35-SW) -> GND
- C55 pad 2: Net-(U35-BOOT) -> +12V
- C56 pad 1: +5V -> GND
- C56 pad 2: Net-(U35-FB) -> Net-(C56-Pad2)
- C57 pad 1: +5V -> GND
- C57 pad 2: Main On/Off Switch -> Net-(U16-IN1+)
- C58 pad 1: +5V -> +3.3V
- C58 pad 2: Main On/Off Switch -> GND
- C59 pad 1: +5V -> GND
- C59 pad 2: Main On/Off Switch -> -12V
- C6 pad 1: Main On/Off Switch -> GND
- C6 pad 2: -12V -> Net-(U1-LDOO)
- C60 pad 1: +5V -> +3.3V
- C60 pad 2: Main On/Off Switch -> GND
- C61 pad 1: Net-(U35-VCC) -> +12V
- C61 pad 2: Main On/Off Switch -> GND
- C62 pad 1: VBUS -> GND
- C62 pad 2: Main On/Off Switch -> -12V
- C63 pad 1: VBUS -> GND
- C63 pad 2: Main On/Off Switch -> +12V
- C64 pad 1: SYS -> Net-(C64-Pad1)
- C64 pad 2: Main On/Off Switch -> Net-(U16-IN2+)
- C65 pad 1: SYS -> SPEAKER SUM BUFF
- C65 pad 2: Main On/Off Switch -> Net-(C64-Pad1)
- C66 pad 1: Net-(U13-VCC) -> Net-(U18-GVDD)
- C66 pad 2: Main On/Off Switch -> GND
- C67 pad 1: Net-(U12-VCC) -> Net-(U19-GVDD)
- C67 pad 2: Main On/Off Switch -> GND
- C68 pad 1: Net-(U12-SW) -> Net-(U18-RINP)
- C68 pad 2: Net-(U12-BOOT) -> TWEET SUM BUFF
- C69 pad 1: +12V -> Net-(U18-RINN)
- C69 pad 2: Net-(U12-FB) -> TWEET SUM BUFF N
- C7 pad 1: Main On/Off Switch -> GND
- C7 pad 2: +12V -> Net-(U1-VNEG)
- C70 pad 1: +12V -> Net-(U18-LINP)
- C70 pad 2: Main On/Off Switch -> WOOF SUM BUFF
- C71 pad 1: +12V -> Net-(U18-LINN)
- C71 pad 2: Main On/Off Switch -> WOOF SUM BUFF N
- C72 pad 1: Main On/Off Switch -> Net-(U19-RINP)
- C72 pad 2: Net-(C72-Pad2) -> SUB SUM BUFF
- C73 pad 1: Main On/Off Switch -> Net-(U19-RINN)
- C73 pad 2: Net-(U24-IN1+) -> SUB SUM BUFF N
- C74 pad 1: SPEAKER SUM BUFF -> +12V
- C74 pad 2: Net-(C74-Pad2) -> GND
- C75 pad 1: Net-(C75-Pad1) -> GND
- C75 pad 2: Net-(U25-IN1+) -> -12V
- C76 pad 1: Net-(C74-Pad2) -> +12V
- C76 pad 2: Net-(U24-IN2+) -> GND
- C77 pad 1: SPEAKER SUM BUFF -> Net-(U19-SYNC)
- C77 pad 2: Net-(C75-Pad1) -> GND
- C78 pad 1: Main On/Off Switch -> GND
- C78 pad 2: Net-(U25-IN2+) -> Net-(C78-Pad2)
- C79 pad 1: Main On/Off Switch -> GND
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Routing:
- added copper zone on B.Cu, net GND
- added copper zone on F.Cu, net GND
- added copper zone on In1.Cu, net GND
- added copper zone on In2.Cu, net GND
Other:
- board outline added: 554.9 x 347.9 mm

Commit message: ñushsh
Parts:
- removed CN1: DIN-504B-M10, lcsc:CONN-TH_DIN-504B-M10
- removed D50: 1N4148WT, Diode_SMD:D_SOD-523
- removed OC1: H11L1, PCM_Package_DIP_AKL:DIP-6_W7.62mm_LongPads
- removed R27: 220, Resistor_SMD:R_0402_1005Metric
- removed R35: 470, Resistor_SMD:R_0402_1005Metric
- moved U25 1068.0 mm to (320.5, 571.6)
- moved C152 1068.0 mm to (308.1, 616.6)
- moved C136 1068.0 mm to (314.8, 570.4)
- moved C128 1068.0 mm to (320.9, 579.3)
- moved C125 1068.0 mm to (321.6, 559.1)
- moved C127 1068.0 mm to (316.6, 573.3)
- moved D55 1068.0 mm to (365.1, 560.4)
- moved R73 1068.0 mm to (321.6, 564.9)
- moved R75 1068.0 mm to (339.8, 561.7)
- moved R78 1068.0 mm to (339.8, 565.6)
- moved R82 1068.0 mm to (311.3, 575.5)
- moved R90 1068.0 mm to (316.1, 584.0)
- moved C126 1068.0 mm to (314.7, 565.1)
- moved C130 1068.0 mm to (312.5, 575.5)
- moved C138 1068.0 mm to (319.7, 575.9)
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Routing:
- removed copper zone on B.Cu, net GND
- removed copper zone on F.Cu, net GND
- removed copper zone on In1.Cu, net GND
- removed copper zone on In2.Cu, net GND
