File: hardware/om-god.kicad_sch (KiCad schematic)
At the start: 0 parts

Commit message: fd
Parts:
- added C1: 100nF, Capacitor_SMD:C_0402_1005Metric, symbol Device:C
- added C44, C55, C59, C60, C61, C62, C70, C71: 10uF, Capacitor_SMD:C_0402_1005Metric, symbol Device:C
- added C45: 22uF, Capacitor_SMD:C_0402_1005Metric, symbol Device:C
- added C56, C65, C66: 1uF, Capacitor_SMD:C_0402_1005Metric, symbol Device:C
- added C57, C69: 4.7uF, Capacitor_SMD:C_0402_1005Metric, symbol Device:C
- added C58: 47nF, Capacitor_SMD:C_0402_1005Metric, symbol Device:C
- added C63, C67, C68: 2.2uF, Capacitor_SMD:C_0402_1005Metric, symbol Device:C
- added C64: 470nF, Capacitor_SMD:C_0402_1005Metric, symbol Device:C
- added CN1: USB-B-Female-90, lcsc:USB-B_TH_USB-B-FEMALE-90, symbol lcsc:USB-B-Female-90
- added CN2, CN3: DIN-504B-M10, lcsc:CONN-TH_DIN-504B-M10, symbol lcsc:DIN-504B-M10
- added CN4: PJ-320D, lcsc:AUDIO-SMD_PJ-320D, symbol lcsc:PJ-320D
- added Card1: TF PUSH, lcsc:TF-SMD_TF-PUSH, symbol lcsc:TFPUSH
- added D1, D10, D11, D12, D13, D14, D15, D16, D17, D18, D19, D2, D20, D21, D22, D23, D24, D25, D3, D4, D5, D50, D51, D52, D53, D54, D55, D56, D57, D58, D59, D6, D60, D61, D62, D63, D64, D65, D66, D67, D68, D69, D7, D70, D71, D72, D8, D9: 1N4148WS_C917117, lcsc:SOD-323_L1.8-W1.3-LS2.5-RD, symbol lcsc:1N4148WS_C917117
- added D26: 1N4148WT, Diode_SMD:D_SOD-523, symbol Diode:1N4148WT
- added D27: PESD15VL1BA, PCM_Diode_SMD_AKL:D_SOD-323_TVS, symbol PCM_Diode_TVS_AKL:PESD15VL1BA
- added FPC1: 5034801200, lcsc:FPC-SMD_5034801200, symbol lcsc:5034801200
- added J1, J2: Conn_01x13_Pin, symbol Connector:Conn_01x13_Pin
- added J3, J4, J5: PJ-625G, lcsc:AUDIO-TH_PJ-625G, symbol lcsc:PJ-625G
- added J6, J7: Conn_01x01_Pin, symbol Connector:Conn_01x01_Pin
- added J8: Conn_01x03, Connector_JST:JST_EH_S3B-EH_1x03_P2.50mm_Horizontal, symbol Connector_Generic:Conn_01x03
- added L4: 1uH, Inductor_SMD:L_0603_1608Metric, symbol Device:L
- added L5, L6: 470nH, Inductor_SMD:L_0603_1608Metric, symbol Device:L
- added L8: EXC14CE900U, linea:FILTER-SMD_4P-L0.9-W0.7-P0.50-BL, symbol linea:EXC14CE900U
- added L9: 470nH, Inductor_SMD:L_Murata_DFE201610P, symbol Device:L
- added Q4: ~, linea:SOT-523-3_L1.6-W0.8-P1.00-LS1.6-BR, symbol DMN313DLT-7:DMN313DLT-7
- added Q5: ~, linea:SOT-363_L2.0-W1.3-P0.65-LS2.1-BL, symbol MMDT2907A-7-F:MMDT2907A-7-F
- added Q6: ~, linea:SOT-23-3_L2.9-W1.3-P1.90-LS2.4-BR, symbol DMP1045U-7:DMP1045U-7
- added R1, R2: 5.1K, Resistor_SMD:R_0402_1005Metric, symbol Device:R
- added R31, R32: 1.5K, Resistor_SMD:R_0402_1005Metric, symbol Device:R
- added R33: 4.7K, Resistor_SMD:R_0402_1005Metric, symbol Device:R
- added R34, R36, R40, R41: 10K, Resistor_SMD:R_0402_1005Metric, symbol Device:R
- added R35: 100, Resistor_SMD:R_0402_1005Metric, symbol Device:R
- added R37: 470, Resistor_SMD:R_0402_1005Metric, symbol Device:R
- added R38: 30.1K, Resistor_SMD:R_0402_1005Metric, symbol Device:R
- added R39: 5.23K, Resistor_SMD:R_0402_1005Metric, symbol Device:R
- added R42: 10m, Resistor_SMD:R_0402_1005Metric, symbol Device:R
- added R43: DNP, Resistor_SMD:R_0402_1005Metric, symbol Device:R
- added R44, R45: 1.5, Resistor_SMD:R_0402_1005Metric, symbol Device:R
- added R46, R47: 3.3, Resistor_SMD:R_0402_1005Metric, symbol Device:R
- added R48, R49: 100K, Resistor_SMD:R_0402_1005Metric, symbol Device:R
- added SW1, SW10, SW11, SW12, SW13, SW14, SW15, SW16, SW17, SW18, SW19, SW2, SW20, SW21, SW22, SW23, SW24, SW25, SW26, SW27, SW28, SW29, SW3, SW30, SW31, SW32, SW33, SW34, SW35, SW36, SW37, SW38, SW39, SW4, SW40, SW41, SW42, SW43, SW44, SW45, SW46, SW47, SW48, SW5, SW56, SW57, SW58, SW6, SW7, SW8, SW9: TS-1003ST-26, lcsc:SW-SMD_4P-L12.0-W12.0-P5.00-LS15.4, symbol lcsc:TS-1003ST-26
- added SW49: RotaryEncoder_Switch, symbol Device:RotaryEncoder_Switch
- added SW50, SW51, SW52, SW53, SW54, SW55: RotaryEncoder, symbol Device:RotaryEncoder
- added TP1, TP2, TP3: TestPoint, TestPoint:TestPoint_Pad_1.5x1.5mm, symbol Connector:TestPoint
- added U1: TDA7297, Package_TO_SOT_THT:TO-220-15_P2.54x2.54mm_StaggerOdd_Lead4.58mm_Vertical, symbol Amplifier_Audio:TDA7297
- added U10, U11, U7, U8, U9: ~, lcsc:SW-TH_6P-L8.0-W8.0-P2.50, symbol lcsc:XKB8080-Z
- added U12: ~, linea:DSBGA-6_L1.4-W1.1-R3-C2-P0.40-BL, symbol LM3281YFQR:LM3281YFQR
- added U13: ~, linea:QFN-24_L4.0-W4.0-P0.50-TL-EP2.7, symbol BQ25896RTWR:BQ25896RTWR
- added U14: ~, linea:DSBGA-9_L1.7-W1.6-R3-C3-P0.50-BL, symbol BQ27220YZFR:BQ27220YZFR
- added U15: FAN48610BUC50X, linea:WLCSP-9_L1.2-W1.2-R3-C3-P0.40-BL, symbol linea:FAN48610BUC50X
- added U16: RS3221-3.3YUTDN4, linea:UTDFN-4_L1.0-W1.0-P0.63-BL-EP-1, symbol linea:RS3221-3.3YUTDN4
- added U17: USBLC6-2P6, Package_TO_SOT_SMD:SOT-666, symbol Power_Protection:USBLC6-2P6
- added U2: TPA3116D2DAD_C2865736, lcsc:HTSSOP-32_L11.0-W6.1-P0.65-LS8.1-BL, symbol lcsc:TPA3116D2DAD_C2865736
- added U3: CY8CMBR3116-LQXIT, lcsc:QFN-24_L4.0-W4.0-P0.50-BL-EP2.6, symbol lcsc:CY8CMBR3116-LQXIT
- added U4: PCM5102APWR, lcsc:TSSOP-20_L6.5-W4.4-P0.65-LS6.4-BL, symbol lcsc:PCM5102APWR
- added U5: HS20HS072RX, lcsc:OLED-SMD_HS20HS072RX, symbol lcsc:HS20HS072RX
- added U6: MKDV4GCL-ABB, lcsc:LGA-8_L6.0-W8.0-P1.27-TL, symbol lcsc:MKDV4GCL-ABB
- added USB2: TYPE-C 16PIN 2MD(073), linea:USB-C-SMD_TYPE-C-6PIN-2MD-073, symbol linea:TYPE-C16PIN2MD(073)
- added VQ: STM32H723ZGT6, lcsc:LQFP-144_L20.0-W20.0-P0.50-LS22.0-BL, symbol lcsc:STM32H723ZGT6
Connections:
- new net: D72.2 (A), SW23.1, SW23.2
- new net: D52.2 (A), SW2.1, SW2.2
- new net: D70.2 (A), SW21.1, SW21.2
- new net: D21.2 (A), SW44.1, SW44.2
- new net: D3.2 (A), SW26.1, SW26.2
- new net: D60.2 (A), SW10.1, SW10.2
- new net: D65.2 (A), SW16.1, SW16.2
- new net: D2.2 (A), SW24.1, SW24.2
- new net: D19.2 (A), SW42.1, SW42.2
- new net: L8.3, U17.6 (I/O1)
- new net: L8.4, U17.4 (I/O2)
- new net: D57.2 (A), SW7.1, SW7.2
- new net: Q5.3 (C2), R48.1
- new net: D24.2 (A), SW47.1, SW47.2
- new net: D63.2 (A), SW14.1, SW14.2
- new net: C68.1, C69.1, C70.1, L6.1, R44.1, R45.1, U12.A1 (FB)
- new net: L5.1, U12.B2 (SW)
- new net: L6.2, R46.2, R47.2
- new net: L5.2, R44.2, R45.2
- new net: D5.2 (A), SW28.1, SW28.2
- new net: D61.2 (A), SW11.1, SW11.2
- new net: D9.2 (A), SW32.1, SW32.2
- new net: D56.2 (A), SW6.1, SW6.2
- new net: D64.2 (A), SW15.1, SW15.2
- new net: D12.2 (A), SW35.1, SW35.2
- new net: L9.2, U15.B1 (SW), U15.B2 (SW)
- new net: D20.2 (A), SW43.1, SW43.2
- new net: D17.2 (A), SW40.1, SW40.2
- new net: R37.2, U13.10 (LIIM)
- new net: J8.2 (Pin_2), R38.2, R39.2, R43.1, TP2.1, U13.11 (TS)
- new net: C61.1, C62.1, C66.1, R42.2, U13.13 (BAT), U13.14 (BAT), U14.C2 (SRN), U16.3 (EN), U16.4 (IN)
- new net: C58.1, L4.1, U13.19 (SW), U13.20 (SW)
- new net: C58.2, U13.21 (BTST)
- new net: C57.1, R39.1, U13.22 (REGN)
- new net: C55.1, U13.23 (PMID)
- new net: R33.1, U13.7 (INT)
- new net: Q4.3 (D), R34.1, U13.8 (OTG)
- new net: D13.2 (A), SW36.1, SW36.2
- new net: Q4.1 (G), R35.1, R36.2
- new net: D62.2 (A), SW12.1, SW12.2
- new net: D55.2 (A), SW5.1, SW5.2
- new net: D51.2 (A), SW25.1, SW25.2
- new net: D16.2 (A), SW39.1, SW39.2
- new net: D23.2 (A), SW46.1, SW46.2
- new net: D7.2 (A), SW30.1, SW30.2
- new net: R2.1, USB2.10 (CC2)
- new net: D11.2 (A), SW34.1, SW34.2
- new net: D68.2 (A), SW19.1, SW19.2
- new net: D14.2 (A), SW37.1, SW37.2
- new net: D15.2 (A), SW38.1, SW38.2
- new net: D8.2 (A), SW31.1, SW31.2
- new net: D54.2 (A), SW4.1, SW4.2
- new net: D53.2 (A), SW3.1, SW3.2
- new net: R40.1, U14.A1 (GPOUT)
- new net: R41.2, U14.B1 (BIN)
- new net: C63.1, C64.1, U14.B3 (VDD)
- new net: D66.2 (A), SW17.1, SW17.2
- new net: D18.2 (A), SW41.1, SW41.2
- new net: D22.2 (A), SW45.1, SW45.2
- new net: D50.2 (A), SW13.1, SW13.2
- new net: D26.2 (A), Q5.2 (B1), Q5.5 (B2)
- new net: Q5.6 (C1), Q6.1 (G), R49.1
- new net: D67.2 (A), SW18.1, SW18.2
- new net: D25.2 (A), SW48.1, SW48.2
- new net: D59.2 (A), SW9.1, SW9.2
- new net: U17.1 (I/O1), USB2.6 (DP1), USB2.8 (DP2)
- new net: U17.3 (I/O2), USB2.5 (DN2), USB2.7 (DN1)
- new net: D1.2 (A), SW1.1, SW1.2
- new net: D10.2 (A), SW33.1, SW33.2
- new net: D58.2 (A), SW8.1, SW8.2
- new net: R1.1, USB2.4 (CC1)
- new net: D6.2 (A), SW29.1, SW29.2
- new net: D71.2 (A), SW22.1, SW22.2
- new net: D69.2 (A), SW20.1, SW20.2
- new net: D4.2 (A), SW27.1, SW27.2
- new net +3.3V: C71.1, R31.2, R32.2, R33.2, R40.2, R46.1, R47.1
- new net +5V: C45.1, U15.A1 (VOUT), U15.A2 (VOUT)
- new net +BATT: C65.1, J8.1 (Pin_1), R42.1, TP1.1, U14.C1 (SRP), U14.C3 (BAT)
- new net 7th: D10.1 (C), D12.1 (C), D14.1 (C), D16.1 (C), D18.1 (C), D2.1 (C), D20.1 (C), D22.1 (C), D24.1 (C), D4.1 (C), D6.1 (C), D8.1 (C)
- new net Chord A: SW1.3, SW1.4, SW11.3, SW11.4, SW24.3, SW24.4, SW26.3, SW26.4
- new net Chord Ab: SW10.3, SW10.4, SW23.3, SW23.4, SW47.3, SW47.4, SW48.3, SW48.4
- new net Chord B: SW14.3, SW14.4, SW25.3, SW25.4, SW29.3, SW29.4, SW30.3, SW30.4
- new net Chord Bb: SW12.3, SW12.4, SW13.3, SW13.4, SW27.3, SW27.4, SW28.3, SW28.4
- new net Chord C: SW15.3, SW15.4, SW2.3, SW2.4, SW31.3, SW31.4, SW32.3, SW32.4
- new net Chord D: SW17.3, SW17.4, SW35.3, SW35.4, SW36.3, SW36.4, SW4.3, SW4.4
- new net Chord Db: SW16.3, SW16.4, SW3.3, SW3.4, SW33.3, SW33.4, SW34.3, SW34.4
- new net Chord E: SW19.3, SW19.4, SW39.3, SW39.4, SW40.3, SW40.4, SW6.3, SW6.4
- new net Chord Eb: SW18.3, SW18.4, SW37.3, SW37.4, SW38.3, SW38.4, SW5.3, SW5.4
- new net Chord F: SW20.3, SW20.4, SW41.3, SW41.4, SW42.3, SW42.4, SW7.3, SW7.4
- new net Chord G: SW22.3, SW22.4, SW45.3, SW45.4, SW46.3, SW46.4, SW9.3, SW9.4
- new net Chord Gb: SW21.3, SW21.4, SW43.3, SW43.4, SW44.3, SW44.4, SW8.3, SW8.4
- new net Extention: D11.1 (C), D13.1 (C), D15.1 (C), D17.1 (C), D19.1 (C), D21.1 (C), D23.1 (C), D25.1 (C), D3.1 (C), D5.1 (C), D7.1 (C), D9.1 (C)
- new net GND: C1.2, C44.2, C45.2, C55.2, C56.2, C57.2, C59.2, C60.2, C61.2, C62.2, C63.2, C64.2, C65.2, C66.2, C67.2, C68.2, C69.2, C70.2, C71.2, D27.1 (K), J8.3 (Pin_3), Q4.2 (S), R1.2, R2.2, R36.1, R37.1, R38.1, R41.1, R43.2, R48.2, R49.2, TP3.1, U12.C2 (GND), U13.17 (PGND), U13.18 (PGND), U13.2 (PSEL), U13.25 (EPAD), U13.9 (CE), U14.B2 (VSS), U15.C1 (PGND), U15.C2 (PGND), U15.C3 (AGND), U16.2 (GND), U16.5 (EP), U17.2 (GND), USB2.1 (GND), USB2.12 (GND), USB2.13 (SHELL), USB2.14 (SHELL)
- new net I2C_SCL: R31.1, U13.5 (SCL), U14.A3 (SCL)
- new net I2C_SDA: R32.1, U13.6 (SDA), U14.A2 (SDA)
- new net LDO_3.3V: U16.1 (OUT)
- new net Mayor: D1.1 (C), D50.1 (C), D51.1 (C), D52.1 (C), D53.1 (C), D54.1 (C), D55.1 (C), D56.1 (C), D57.1 (C), D58.1 (C), D59.1 (C), D60.1 (C)
- new net Minor: D61.1 (C), D62.1 (C), D63.1 (C), D64.1 (C), D65.1 (C), D66.1 (C), D67.1 (C), D68.1 (C), D69.1 (C), D70.1 (C), D71.1 (C), D72.1 (C)
- new net RESET: U13.12 (QON)
- new net SYS: C44.1, C59.1, C60.1, C67.1, L4.2, L9.1, R34.2, U12.A2 (VIN), U12.B1 (MODE), U12.C1 (EN), U13.15 (SYS), U13.16 (SYS), U15.A3 (VIN), U15.B3 (EN)
- new net USB_5V: C56.1, Q5.4 (E2), Q6.2 (S), U13.1 (VBUS)
- new net VBUS: C1.1, D26.1 (K), D27.2 (A), Q5.1 (E1), Q6.3 (D), R35.2, U17.5 (VBUS), USB2.11 (VBUS), USB2.2 (VBUS)
- no-connect marks 0 -> 3
Other:
- note added: "Advanced Funtionalities"
- note added: "Audio Amplifiers"
- note added: "Audio Out"
- note added: "Chord Matrix"
- note added: "Chords Volume"
- note added: "DAC"
- note added: "DIN-MIDI"
- note added: "External Micro SD Card"
- note added: "Function Knob"
- note added: "Headphones Out"
- note added: "I/O"
- note added: "If using thermistor, remove R43"
- note added: "Instant Off"
- note added: "Keyboard Volume"
- note added: "Main"
- note added: "Main Buttons"
- note added: "Main Knobs"
- note added: "Main Volume"
- note added: "Metronome"
- note added: "Midi"
- note added: "NAnd Flash"
- note added: "Next Chord"
- note added: "Octave Down"
- note added: "Octave Up"
- note added: "On/Off"
- note added: "Pedal"
- note added: "Power Managment"
- note added: "Recording"
- note added: "Recording Mode"
- note added: "Rythm"
- note added: "Rythm Volume"
- note added: "Sonic Strings"
- note added: "Stereo Out"
- note added: "Sustain Chord"
- note added: "Touch Pad"
- note added: "Touch Pad Volume"
- note added: "USB-MIDI"
- note added: "Usb Power outlet / Coding"
- note added: "VQ"
- note added: "Vibrato Knob"
- note added: "Volume"

Commit message: yes
Parts:
- removed CN4: PJ-320D, lcsc:AUDIO-SMD_PJ-320D, symbol lcsc:PJ-320D
- removed D26: 1N4148WT, Diode_SMD:D_SOD-523, symbol Diode:1N4148WT
- removed J2: Conn_01x13_Pin, symbol Connector:Conn_01x13_Pin
- removed J6, J7: Conn_01x01_Pin, symbol Connector:Conn_01x01_Pin
- removed J8: Conn_01x03, Connector_JST:JST_EH_S3B-EH_1x03_P2.50mm_Horizontal, symbol Connector_Generic:Conn_01x03
- removed L9: 470nH, Inductor_SMD:L_Murata_DFE201610P, symbol Device:L
- removed Q4: ~, linea:SOT-523-3_L1.6-W0.8-P1.00-LS1.6-BR, symbol DMN313DLT-7:DMN313DLT-7
- removed Q5: ~, linea:SOT-363_L2.0-W1.3-P0.65-LS2.1-BL, symbol MMDT2907A-7-F:MMDT2907A-7-F
- removed Q6: ~, linea:SOT-23-3_L2.9-W1.3-P1.90-LS2.4-BR, symbol DMP1045U-7:DMP1045U-7
- removed TP1, TP2, TP3: TestPoint, TestPoint:TestPoint_Pad_1.5x1.5mm, symbol Connector:TestPoint
- removed U1: TDA7297, Package_TO_SOT_THT:TO-220-15_P2.54x2.54mm_StaggerOdd_Lead4.58mm_Vertical, symbol Amplifier_Audio:TDA7297
- removed U12: ~, linea:DSBGA-6_L1.4-W1.1-R3-C2-P0.40-BL, symbol LM3281YFQR:LM3281YFQR
- removed U13: ~, linea:QFN-24_L4.0-W4.0-P0.50-TL-EP2.7, symbol BQ25896RTWR:BQ25896RTWR
- removed U14: ~, linea:DSBGA-9_L1.7-W1.6-R3-C3-P0.50-BL, symbol BQ27220YZFR:BQ27220YZFR
- removed U15: FAN48610BUC50X, linea:WLCSP-9_L1.2-W1.2-R3-C3-P0.40-BL, symbol linea:FAN48610BUC50X
- removed U16: RS3221-3.3YUTDN4, linea:UTDFN-4_L1.0-W1.0-P0.63-BL-EP-1, symbol linea:RS3221-3.3YUTDN4
- removed U4: PCM5102APWR, lcsc:TSSOP-20_L6.5-W4.4-P0.65-LS6.4-BL, symbol lcsc:PCM5102APWR
- added AUDIO1: PJ-393_C2837065, lcsc:AUDIO-SMD_PJ-393, symbol lcsc:PJ-393_C2837065
- added C10, C104, C12, C133, C134, C135, C136, C142, C143, C145, C146, C148, C155, C156, C157, C158, C167, C177, C179, C180, C181, C185, C186, C189, C19, C194, C20, C3, C4, C41, C42, C43, C46, C47, C48, C49, C5, C51, C52, C53, C54, C6, C7, C8, C82, C83, C84, C86, C9, C94, C96: 0.1uF, symbol Device:C
- added C105, C106, C107, C120, C121, C124, C127, C128, C166, C22, C23, C24, C32, C33, C34, C35, C50, C95: 1uF, symbol Device:C
- added C108, C109, C21, C25, C38: 1nF, symbol Device:C
- added C11, C18, C188, C191, C195, C196, C2, C80, C81, C85, C92, C93, C97: 2.2uF, symbol Device:C
- added C110, C111, C112, C113, C165, C28, C29, C30, C31: 220nF, symbol Device:C
- added C114, C115, C131, C26, C39: 100nF, symbol Device:C
- added C116, C117, C27, C40: 220uF, symbol Device:C_Polarized
- added C118, C119, C125, C126: 680nF, symbol Device:C
- added C122, C123, C129, C130, C132, C36, C37: 10nF, symbol Device:C
- added C13, C14, C147, C15, C150, C152, C153, C16, C17, C184, C187, C190, C192, C193, C87, C88, C89, C90, C91: 10uF, symbol Device:C_Polarized
- added C137, C138: 220pF, Capacitor_SMD:C_0402_1005Metric, symbol Device:C
- added C139: 0.1uF, Capacitor_SMD:C_0402_1005Metric, symbol Device:C
- added C140, C149, C151: 1uF, symbol Device:C_Polarized
- added C141: 0.056uF, symbol Device:C_Polarized
- added C144: 2.2uF, symbol Device:C_Polarized
- added C154: 22pF, symbol Device:C
- added C159, C168: 47pF, symbol Device:C
- added C160, C161, C162, C163, C169, C170, C171, C172, C173, C174, C182, C183: 22uF, symbol Device:C
- added C164, C175, C176, C178: 10uF, symbol Device:C
- added C72, C73, C75, C77: 82nF, PCM_Capacitor_THT_AKL:C_Rect_L4.0mm_W2.5mm_P2.50mm, symbol PCM_Capacitor_AKL:C_Rect_L4.0mm_W2.5mm_P2.50mm
- added C74, C76, C78, C79: 5.6nF, PCM_Capacitor_THT_AKL:C_Rect_L4.0mm_W2.5mm_P2.50mm, symbol PCM_Capacitor_AKL:C_Rect_L4.0mm_W2.5mm_P2.50mm
- added D28: BAT54, PCM_Package_TO_SOT_SMD_AKL:SOT-23, symbol PCM_Diode_Schottky_AKL:BAT54
- added D29, D30, D31: LED, symbol Device:LED
- added J2: Conn_01x03_Pin, symbol Connector:Conn_01x03_Pin
- added L1, L10, L11, L2, L3, L7: 10uH, symbol Device:L
- added L12: 6.8uH, Inductor_SMD:L_6.3x6.3_H3, symbol Device:L
- added L13: 6.8uH, symbol Device:L
- added L14: 15uH, symbol Device:L
- added Q1, Q2, Q3: Si7617DN, Package_SO:Vishay_PowerPAK_1212-8_Single, symbol Transistor_FET:Si7617DN
- added R10, R13, R17, R18, R26: 100k, symbol Device:R
- added R100, R101, R87, R99: 10K, Resistor_SMD:R_0402_1005Metric, symbol Device:R
- added R102, R66, R69, R74: 100K, Resistor_SMD:R_0402_1005Metric, symbol Device:R
- added R103: NTCG163JF103FT1S, lcsc:R0603, symbol lcsc:NTCG163JF103FT1S
- added R104: 9.31K, Resistor_SMD:R_0402_1005Metric, symbol Device:R
- added R105: 430K, Resistor_SMD:R_0402_1005Metric, symbol Device:R
- added R11, R16: 75k, symbol Device:R
- added R12, R9: 47k, symbol Device:R
- added R14, R15, R19, R20, R24, R25: 3.3, symbol Device:R
- added R21, R22, R27, R28, R29, R30, R50, R51, R52, R53, R7, R8, R82, R83, R84, R85: 10K, symbol Device:R
- added R23: 10k, symbol Device:R
- added R3, R4: 470K, symbol Device:R
- added R5, R59, R6, R60, R61, R62, R63, R64, R65, R67, R68, R70, R71, R72, R73, R75: 6K, symbol Device:R
- added R58: 200K, Resistor_SMD:R_0402_1005Metric, symbol Device:R
- added R76, R77, R78, R79, R80, R81, R89, R94: 1K, symbol Device:R
- added R86: 22.1K, Resistor_SMD:R_0402_1005Metric, symbol Device:R
- added R88: 32.4K, Resistor_SMD:R_0402_1005Metric, symbol Device:R
- added R90, R95, R98: 100K, symbol Device:R
- added R91: 10, symbol Device:R
- added R92: 2, symbol Device:R
- added R93, R96: 0.01, symbol Device:R
- added R97: 500K, symbol Device:R
- added U1, U18, U19, U20, U22, U24, U25, U28, U29: NE5532DR, lcsc:SOIC-8_L4.9-W3.9-P1.27-LS6.0-BL, symbol lcsc:NE5532DR
- added U12, U13, U14, U35: LMR33630ADDAR, lcsc:ESOP-8_L4.9-W3.9-P1.27-LS6.0-TL-EP, symbol lcsc:LMR33630ADDAR
- added U15: TPS54202DDC, Package_TO_SOT_SMD:SOT-23-6, symbol Regulator_Switching:TPS54202DDC
- added U16, U26, U4: PCM5122PW, Package_SO:TSSOP-28_4.4x9.7mm_P0.65mm, symbol Audio:PCM5122PW
- added U21: TPA6120A2DWP, lcsc:HSOP-20_L12.8-W7.5-P1.27-LS10.3-BL-EP3.3, symbol lcsc:TPA6120A2DWP
- added U23: TS5A23159RSER, lcsc:UQFN-10_L2.0-W1.5-P0.50-BL-EP, symbol lcsc:TS5A23159RSER
- added U30: TPA3116D2DAD_C2865736, lcsc:HTSSOP-32_L11.0-W6.1-P0.65-LS8.1-BL, symbol lcsc:TPA3116D2DAD_C2865736
- added U31: BQ24610, Package_DFN_QFN:VQFN-24-1EP_4x4mm_P0.5mm_EP2.45x2.45mm, symbol Battery_Management:BQ24610
- added U32: TUSB422IYFPR, lcsc:DSBGA-9_L1.4-W1.3-R3-C3-P0.40-BL, symbol lcsc:TUSB422IYFPR
- added U33, U34: SIS412DN-T1-GE3-ES, lcsc:PDFN-8_L3.1-W3.1-P0.65-LS3.4-BL, symbol lcsc:SIS412DN-T1-GE3-ES
- C44, C66: footprint Capacitor_SMD:C_0402_1005Metric -> (none)
- C45: value 22uF -> 220nF; footprint Capacitor_SMD:C_0402_1005Metric -> (none)
- C55: value 10uF -> 0.1uF; footprint Capacitor_SMD:C_0402_1005Metric -> (none)
- C56: value 1uF -> 47pF; footprint Capacitor_SMD:C_0402_1005Metric -> (none); now not fitted
- C57: value 4.7uF -> 22uF; footprint Capacitor_SMD:C_0402_1005Metric -> (none)
- C58: value 47nF -> 22uF; footprint Capacitor_SMD:C_0402_1005Metric -> (none)
- C59, C60, C70, C71: value 10uF -> 22uF; footprint Capacitor_SMD:C_0402_1005Metric -> (none)
- C61: value 10uF -> 1uF; footprint Capacitor_SMD:C_0402_1005Metric -> (none)
- C62: value 10uF -> 220nF; footprint Capacitor_SMD:C_0402_1005Metric -> (none)
- C63: value 2.2uF -> 10uF; footprint Capacitor_SMD:C_0402_1005Metric -> (none)
- C64: value 470nF -> 10uF; footprint Capacitor_SMD:C_0402_1005Metric -> (none)
- C65: value 1uF -> 220nF; footprint Capacitor_SMD:C_0402_1005Metric -> (none)
- C67: value 2.2uF -> 1uF; footprint Capacitor_SMD:C_0402_1005Metric -> (none)
- C68: value 2.2uF -> 0.1uF; footprint Capacitor_SMD:C_0402_1005Metric -> (none)
- C69: value 4.7uF -> 47pF; footprint Capacitor_SMD:C_0402_1005Metric -> (none); now not fitted
- L4: value 1uH -> 8uH; footprint Inductor_SMD:L_0603_1608Metric -> (none)
- L5: value 470nH -> 15uH; footprint Inductor_SMD:L_0603_1608Metric -> (none)
- L6: value 470nH -> 27uH; footprint Inductor_SMD:L_0603_1608Metric -> (none)
- R1, R2: value 5.1K -> 1.5K
- R31: value 1.5K -> 100K
- R32: value 1.5K -> 24.9K
- R33: value 4.7K -> 100K
- R34, R40, R41: value 10K -> 100K
- R35: value 100 -> 100K
- R36: value 10K -> 43.2K
- R37: value 470 -> 100K
- R38: value 30.1K -> 100K
- R39: value 5.23K -> 9.09K
- R42: value 10m -> 9.09K
- R43: value DNP -> 49.9
- R44: value 1.5 -> 50k
- R45: value 1.5 -> 2.61k
- R46, R47: value 3.3 -> 470K; footprint Resistor_SMD:R_0402_1005Metric -> (none)
- R48, R49: value 100K -> 470K; footprint Resistor_SMD:R_0402_1005Metric -> (none)
- renumbered VQ to VQ1
Connections:
- net I2C_SDA is gone; now on net GND: R32.1
- net USB_5V is gone; now on net +5V: C56.1
- net +3.3V: now also R1.1, R2.2, R35.2, U3.7 (VDD), C139.1, C15.1, C159.1, C160.1, C161.1, C162.1, C163.1, C184.1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; no longer C71.1, R31.2, R32.2, R33.2, R40.2, R46.1, R47.1
- net +5V: now also C57.1, C58.1, C59.1, C60.1, L4.2, R31.2; no longer C45.1
- net +BATT: now also C152.1, C153.1, C154.2, C155.1, Q3.5 (D), R96.2, R97.1, U31.13 (SRN); no longer C65.1, R42.1
- net GND: now also C58.2, J3.2, J4.2, L6.2, R39.1, R42.1, U2.1 (MODSEL), U2.10 (LINP), U2.11 (LINN), U2.13 (AM2), U2.14 (AM1), U2.15 (AM0)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; no longer C55.2, C56.2, C68.2, C69.2, R1.2, R2.2, R37.1, R38.1, R41.1, R48.2, R49.2
- net SYS: now also C45.1, C62.1, C63.1, C64.1, C65.1, C145.2, C147.1, C148.2, C150.1, C164.1, C165.1, Q3.1 (S)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; no longer C59.1, C60.1, C67.1, L4.2, R34.2
- net VBUS: now also Q1.5 (D), R100.2, R101.2, R92.2, R99.2, U32.A2 (VBUSIN); no longer R35.2
- net DN USB: now reaches L8.1
- net DP USB: now reaches L8.2
- net at R48.1: now also U26.6 (OUTL)
- net at L5.1: now also C68.1, U12.8 (SW)
- net STEREO BUFF L/MONO: now reaches J4.6
- net STEREO BUFF L/MONO: now also U23.10 (COM1)
- net STEREO GPIO L/MONO: now reaches J4.7
- net STEREO GPIO L/MONO: now also R83.2
- net PG: now reaches R37.2
- net PG: now also R33.2, R34.2, R40.2, U12.4 (PG), U13.4 (PG), U14.4 (PG), U35.4 (PG)
- net at L4.1: now also C55.1, U35.8 (SW); no longer C58.1
- net at R33.1: now also C61.1, U35.6 (VCC)
- net at R34.1: now also C66.1, U13.6 (VCC)
- net at R35.1, R36.2: now also C159.2, U13.5 (FB)
- net STEREO BUFF R: now reaches J3.6
- net STEREO BUFF R: now also U1.2 (OUT2), U1.3 (IN2-)
- net STEREO GPIO R: now reaches J3.7
- net STEREO GPIO R: now also R82.2
- net at USB2.10 (CC2): now also C137.1, U32.A1 (CC2); no longer R2.1
- net MUTE SUB: now reaches U2.12 (MUTE)
- net MUTE SUB: now also R10.1
- net at U2.16 (SYNC): now also C21.1, R23.2
- net +12V: now reaches U2.17 (AVCC)
- net +12V: now also C69.1, C70.1, C71.1, L5.2, R38.2, R41.2, U2.18 (PVCC), U2.19 (PVCC), U2.31 (PVCC), U2.32 (PVCC), C104.2, C108.2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
- net /SD SUB: now reaches U2.2 (SDZ)
- net /SD SUB: now also U2.3 (FAULTZ), R13.2
- net at U2.20 (BSNL): now also C30.1
- net at U2.21 (OUTNL): now also U2.23 (OUTPL), C30.2, C31.1, L2.1
- net at U2.24 (BSPL): now also C31.2
- net at U2.26 (BSNR): now also C29.2
- net at U2.27 (OUTNR): now also U2.29 (OUTPR), C28.1, C29.1, L1.1
- net at U2.30 (BSPR): now also C28.2
- net at U2.4 (RINP): now also C24.1
- net at U2.5 (RINN): now also C23.1
- net at U2.6 (PLIMIT): now also U2.7 (GVDD), C22.1, R12.1
- net at U2.8 (GAIN/SLV): now also R11.1, R12.2
- net at R40.1: now also C67.1, U12.6 (VCC)
- net at R49.1: now also U26.7 (OUTR)
- net SS 0: now reaches J1.1 (Pin_1)
- new net: R80.1, U21.16 (RIN-)
- new net: R79.2, R81.2, U21.17 (RIN+)
- new net: R76.2, R77.2, U21.4 (LIN+)
- new net: R78.1, U21.5 (LIN-)
- new net: U31.19 (LODRV), U34.4 (G)
- new net: C143.2, L12.1, U31.20 (PH), U33.1 (S), U33.2 (S), U33.3 (S), U34.5 (D), U34.6 (D), U34.7 (D), U34.8 (D), U34.9 (D)
- new net: C123.1, R20.1
- new net: C140.1, U31.10 (VREF), U31.4 (CE)
- new net: R66.1, R86.1, U31.11 (ISET1)
- new net: C154.1, R97.2, R98.1, U31.12 (VFB)
- new net: C155.2, C156.1, L12.2, R96.1, U31.14 (SRP)
- new net: R69.1, R87.1, U31.15 (ISET2)
- new net: R74.1, R88.1, U31.16 (ACSET)
- new net: C149.1, D28.1 (A), U31.18 (REGN)
- new net: C145.1, C146.2, Q2.1 (S), Q2.2 (S), Q2.3 (S), R93.1, U31.2 (ACP)
- new net: U31.21 (HIDRV), U33.4 (G)
- new net: C143.1, D28.3 (K), U31.22 (BTST)
- new net: R94.1, U31.23 (~{BATDRV})
- new net: C151.1, R91.2, U31.24 (VCC)
- new net: R89.2, U31.3 (~{ACDRV})
- new net: D29.1 (K), U31.5 (STAT1)
- new net: C157.1, R102.2, U31.6 (TS)
- new net: C141.1, U31.7 (TTC)
- new net: D31.1 (K), U31.8 (~{PG})
- new net: D30.1 (K), U31.9 (STAT2)
- new net: C186.2, C187.1, U16.26 (LDOO)
- new net: R60.1, R61.1, U19.6 (IN1+)
- new net: R47.1, U16.6 (OUTL)
- new net: C68.2, U12.7 (BOOT)
- new net: C75.1, C77.2, R51.2
- new net: R64.1, R67.2, U28.3 (IN2-)
- new net: R72.1, R75.2, U29.3 (IN2-)
- new net: C167.1, L14.1, U14.8 (SW)
- new net: C76.2, R50.2, U24.4 (IN2+)
- new net: C73.2, R28.1, U24.6 (IN1+)
- new net: D30.2 (A), R100.1
- new net: C69.2, R41.1, R42.2, U12.5 (FB)
- new net: C55.2, U35.7 (BOOT)
- new net: C180.1, L6.1, U15.2 (SW)
- new net: C180.2, U15.6 (BOOT)
- new net: R62.2, R63.1, U19.7 (IN1-)
- new net: C72.2, R27.1, R28.2
- new net: C84.2, C90.1, U26.26 (LDOO)
- new net: C110.1, L3.1, U30.29 (OUTPR)
- new net: R23.1, U30.16 (SYNC)
- new net: C131.2, R26.1
- new net: C122.2, R19.2
- new net: C74.2, C76.1, R29.2
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Other:
- note added: "Connect int a gpio exti"
- note removed: "Audio Amplifiers"
- note removed: "DAC"
- note removed: "If using thermistor, remove R43"
- note removed: "Touch Pad"
- note removed: "Usb Power outlet / Coding"
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
Commit message: g
Parts:
- removed U6: MKDV4GCL-ABB, lcsc:LGA-8_L6.0-W8.0-P1.27-TL, symbol lcsc:MKDV4GCL-ABB
Other:
- note removed: "NAnd Flash"
Changed lines of the file:
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@@
 		)
 	)
-	(text "NAnd Flash"
-		(exclude_from_sim no)
-		(at 1071.118 378.46 0)
-		(effects
-			(font
-				(size 1.27 1.27)
-			)
-		)
-	)
 	(text "Function Knob"
 		(exclude_from_sim no)
@@
 		)
 	)
-	(polyline
-		(pts
-			(xy 1056.64 405.13) (xy 1056.64 381)
-		)
-		(stroke
-			(width 0)
-			(type default)
-		)
-	)
 	(wire
 		(pts
@@
 		)
 	)
-	(polyline
-		(pts
-			(xy 1056.64 381) (xy 1087.12 381)
-		)
-		(stroke
-			(width 0)
-			(type default)
-		)
-	)
 	(wire
 		(pts
@@
 		)
 	)
-	(polyline
-		(pts
-			(xy 1087.12 382.27) (xy 1087.12 405.13)
-		)
-		(stroke
-			(width 0)
-			(type default)
-		)
-	)
 	(wire
 		(pts
@@
 		)
 	)
-	(polyline
-		(pts
-			(xy 1087.12 381) (xy 1087.12 383.54)
-		)
-		(stroke
-			(width 0)
-			(type default)
-		)
-	)
 	(wire
 		(pts
@@
 		)
 	)
-	(polyline
-		(pts
-			(xy 1087.12 405.13) (xy 1056.64 405.13)
-		)
-		(stroke
-			(width 0)
-			(type default)
-		)
-	)
 	(wire
 		(pts
@@
 					(unit 1)
 				)
-			)
-		)
-	)
-	(symbol
-		(lib_id "lcsc:MKDV4GCL-ABB")
-		(at 1071.88 396.24 0)
-		(unit 1)
-		(exclude_from_sim no)
-		(in_bom yes)
-		(on_board yes)
-		(dnp no)
-		(fields_autoplaced yes)
-		(property "Reference" "U6"
-			(at 1071.88 384.81 0)
-			(effects
-				(font
-					(size 1.27 1.27)
-				)
-			)
-		)
-		(property "Value" "MKDV4GCL-ABB"
-			(at 1071.88 387.35 0)
-			(effects
-				(font
-					(size 1.27 1.27)
-				)
-			)
-		)
-		(property "Footprint" "lcsc:LGA-8_L6.0-W8.0-P1.27-TL"
-			(at 1071.88 407.67 0)
-			(effects
-				(font
-					(size 1.27 1.27)
-				)
-				(hide yes)
-			)
-		)
-		(property "Datasheet" ""
-			(at 1071.88 396.24 0)
-			(effects
-				(font
-					(size 1.27 1.27)
-				)
-				(hide yes)
-			)
-		)
-		(property "Description" ""
-			(at 1071.88 396.24 0)
-			(effects
-				(font
-					(size 1.27 1.27)
-				)
-				(hide yes)
-			)
-		)
-		(property "LCSC Part" "C7500178"
-			(at 1071.88 410.21 0)
-			(effects
-				(font
-					(size 1.27 1.27)
-				)
-				(hide yes)
-			)
-		)
-		(pin "1"
-		)
-		(pin "6"
-		)
-		(pin "5"
-		)
-		(pin "3"
-		)
-		(pin "8"
-		)
-		(pin "4"
-		)
-		(pin "7"
-		)
-		(pin "2"
-		)
-		(instances
-			(project ""
-				(path "/0dd47ee7-841f-4fd7-9fd1-ca99fc50fdde"
-					(reference "U6")
-					(unit 1)
-				)

Commit message: yes
Parts:
- removed CN1: USB-B-Female-90, lcsc:USB-B_TH_USB-B-FEMALE-90, symbol lcsc:USB-B-Female-90
- added C100, C98, C99: 0.1uF, Capacitor_SMD:C_0402_1005Metric, symbol Device:C
- added C101, C102, C103, C197, C198, C199, C200, C201, C202, C203, C204, C205, C207, C210, C211: 100nF, Capacitor_SMD:C_0402_1005Metric, symbol Device:C
- added C206: 4.7uF, Capacitor_SMD:C_0402_1005Metric, symbol Device:C
- added C208, C209: 2.2uF, Capacitor_SMD:C_0402_1005Metric, symbol Device:C
- added C212: 100uF, Capacitor_SMD:C_0402_1005Metric, symbol Device:C
- added C213, C214: 5.6pF, Capacitor_SMD:C_0402_1005Metric, symbol Device:C
- added C215, C216: 5.1pF, Capacitor_SMD:C_0402_1005Metric, symbol Device:C
- added D26: 1N4148WT, Diode_SMD:D_SOD-523, symbol Diode:1N4148WT
- added D32: SB520, PCM_Diode_THT_AKL:D_DO-201AD_P12.70mm_Horizontal, symbol PCM_Diode_Schottky_AKL:SB520
- added J10, J8, J9: Conn_01x02_Socket, lcsc:CONN-TH_2P-P5.00_WJ500V-5.08-2P, symbol Connector:Conn_01x02_Socket
- added J11, J6: Conn_01x08_Pin, lcsc:CONN-TH_B8PS-VH-LF-SN, symbol Connector:Conn_01x08_Pin
- added OC1: H11L1, PCM_Package_DIP_AKL:DIP-6_W7.62mm_LongPads, symbol PCM_Optocoupler_Logic_AKL:H11L1
- added R106, R107, R108, R109, R110, R55, R56, R57: 22, Resistor_SMD:R_0402_1005Metric, symbol Device:R
- added R111, R112, R113, R114, R115, R116, R127: 10K, Resistor_SMD:R_0402_1005Metric, symbol Device:R
- added R117, R118: 0, Resistor_SMD:R_0402_1005Metric, symbol Device:R
- added R119, R121, R126: 10k, Resistor_SMD:R_0402_1005Metric, symbol Device:R
- added R120: 4.7k, Resistor_SMD:R_0402_1005Metric, symbol Device:R
- added R122, R54: 1k, Resistor_SMD:R_0402_1005Metric, symbol Device:R
- added R123: 220, Resistor_SMD:R_0402_1005Metric, symbol Device:R
- added R124: 33, Resistor_SMD:R_0402_1005Metric, symbol Device:R
- added R125: 10, Resistor_SMD:R_0402_1005Metric, symbol Device:R
- added SW59, SW60: SW_Push, Button_Switch_SMD:SW_SPST_CK_RS282G05A3, symbol Switch:SW_Push
- added U27, U36: FPC-05F-6PH20, lcsc:FPC-SMD_6P-P0.50_XUNPU_FPC-05F-6PH20, symbol lcsc:FPC-05F-6PH20
- added U37: ~, lcsc:CRYSTAL-SMD_4P-L3.2-W2.5-BL_SIT8008BI, symbol lcsc:CRYSTAL
- added U6: W29N02KVSIAF, lcsc:TSOP-48_L12.0-W18.4-P0.50-LS20.0-TL, symbol lcsc:W29N02KVSIAF
- added Y2: 32.768KHz, lcsc:FC-135R_L3.2-W1.5, symbol Device:Crystal
- C10, C104, C105, C106, C107, C108, C109, C11, C110, C111, C112, C113, C114, C115, C118, C119, C12, C120, C121, C122, C123, C124, C125, C126, C127, C128, C129, C130, C131, C132, C133, C134, C135, C136, C142, C143, C145, C146, C148, C154, C155, C156, C157, C158, C159, C166, C167, C168, C173, C174, C175, C176, C177, C178, C179, C18, C180, C181, C182, C183, C185, C186, C188, C189, C19, C191, C194, C195, C196, C2, C20, C21, C22, C23, C24, C25, C26, C28, C29, C3, C30, C31, C32, C33, C34, C35, C36, C37, C38, C39, C4, C41, C42, C45, C46, C47, C48, C49, C5, C50, C51, C52, C53, C54, C55, C56, C6, C61, C66, C67, C68, C7, C71, C8, C80, C81, C82, C83, C84, C85, C86, C9, C92, C93, C94, C95, C96, C97: footprint (none) -> Capacitor_SMD:C_0402_1005Metric
- C116, C117, C13, C14, C147, C15, C150, C152, C153, C16, C17, C184, C187, C190, C192, C193, C27, C40, C87, C88, C89, C90, C91: footprint (none) -> Capacitor_THT:CP_Radial_D8.0mm_P3.50mm
- C140, C149, C151: footprint (none) -> Capacitor_THT:CP_Radial_D5.0mm_P2.00mm
- C141: value 0.056uF -> 0.1uF; footprint (none) -> Capacitor_THT:CP_Radial_D5.0mm_P2.00mm
- C144: footprint (none) -> Capacitor_THT:CP_Radial_D8.0mm_P2.50mm
- C160, C161, C162, C163, C164, C165, C169, C170, C171, C172, C43, C44, C57, C58, C59, C60, C62, C63, C64, C65, C69, C70: footprint (none) -> Capacitor_SMD:C_0603_1608Metric
- C72, C73: footprint PCM_Capacitor_THT_AKL:C_Rect_L4.0mm_W2.5mm_P2.50mm -> Capacitor_SMD:C_0603_1608Metric
- D29, D30, D31: footprint (none) -> LED_SMD:LED_0603_1608Metric
- J1: footprint (none) -> Connector_PinHeader_2.54mm:PinHeader_1x13_P2.54mm_Vertical
- J2: footprint (none) -> Connector_PinHeader_2.54mm:PinHeader_1x03_P2.54mm_Vertical
- L1, L10, L11, L2, L3, L7: footprint (none) -> lcsc:IND-SMD_L11.0-W10.5_SL1050-330M
- L13: footprint (none) -> lcsc:IND-SMD_L3.2-W2.5_L3225
- L14, L5: footprint (none) -> lcsc:IND-SMD_L12.3-W12.3
- L4: footprint (none) -> lcsc:L1206
- L6: footprint (none) -> lcsc:IND-SMD_L4.8-W3.4
- L8: footprint linea:FILTER-SMD_4P-L0.9-W0.7-P0.50-BL -> lcsc:FILTER-SMD_4P-L0.9-W0.7-P0.50-BL
- R10, R11, R12, R13, R14, R15, R16, R17, R18, R19, R20, R21, R22, R23, R24, R25, R26, R27, R28, R29, R3, R30, R4, R46, R47, R48, R49, R5, R50, R51, R52, R53, R59, R6, R60, R61, R62, R63, R64, R65, R67, R68, R7, R70, R71, R72, R73, R75, R76, R77, R78, R79, R8, R80, R81, R82, R83, R84, R85, R89, R9, R90, R91, R92, R93, R94, R95, R96, R97, R98: footprint (none) -> Resistor_SMD:R_0402_1005Metric
- SW49: footprint (none) -> lcsc:SW-TH_EC11E1820402; LCSC (none) -> C361165
- SW50, SW51, SW52, SW53, SW54, SW55: footprint (none) -> lcsc:SW-TH_EC12EXXXX; LCSC (none) -> C470684
- U10, U11, U7, U8, U9: footprint lcsc:SW-TH_6P-L8.0-W8.0-P2.50 -> lcsc:SW-TH_6P-L7.0-W7.0-P2.00_7-7-ZS; LCSC (none) -> C5379891
- U5: Name OLED -> (none)
- USB2: footprint linea:USB-C-SMD_TYPE-C-6PIN-2MD-073 -> lcsc:USB-C-SMD_TYPE-C-6PIN-2MD-073
Connections:
- net ADR1 HEADPHONE is gone; now on net GND: U4.24 (ADR1/MISO/FMT)
- net ADR1 SPEAKER is gone; now on net GND: U16.24 (ADR1/MISO/FMT)
- net ADR1 STEREO OUT is gone; now on net GND: U26.24 (ADR1/MISO/FMT)
- net ADR2 HEADPHONE is gone; now on net GND: U4.16 (ADR2/GPIO2/DOUT)
- net ADR2 SPEAKER is gone; now on net GND: U16.16 (ADR2/GPIO2/DOUT)
- net ADR2 STEREO OUT is gone; now on net GND: U26.16 (ADR2/GPIO2/DOUT)
- net SCL HEADPHONE is gone; now on net SCL I2C2: U4.12 (SCL/MC/ATT1)
- net SCL SPEAKER is gone; now on net SCL I2C1: U16.12 (SCL/MC/ATT1)
- net SCL STEREO OUT is gone; now on net SCL I2C4: U26.12 (SCL/MC/ATT1)
- net SDA HEADPHONE is gone; now on net SDA I2C2: U4.11 (SDA/MOSI/ATT2)
- net SDA SPEAKER is gone; now on net SDA I2C1: U16.11 (SDA/MOSI/ATT2)
- net SDA STEREO OUT is gone; now on net SDA I2C4: U26.11 (SDA/MOSI/ATT2)
- net SS SCL is gone; now on net SCL I2C1: U3.22 (I2CSCL)
- net SS SDA is gone; now on net SDA I2C1: U3.21 (I2CSDA)
- net +12V: now also J11.1 (Pin_1), J11.2 (Pin_2), J6.1 (Pin_1), J6.2 (Pin_2)
- net +3.3V: now also Card1.4 (VDD), FPC1.11, FPC1.8, FPC1.9, VQ1.108 (VDD), VQ1.121 (VDD), VQ1.131 (VDD), VQ1.144 (VDD), VQ1.17 (VDD), VQ1.30 (VDD), VQ1.35 (PA1), VQ1.39 (VDD)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
- net +3.3VA: now also VQ1.32 (VREF+), VQ1.33 (VDDA), C101.1, R117.1, R117.2, R118.2
- net +5V: now also J11.6 (Pin_6), J6.6 (Pin_6), R120.2
- net -12V: now also J11.7 (Pin_7), J6.7 (Pin_7)
- net 7th: now also VQ1.37 (PA3)
- net BCK HEADPHONE: now also VQ1.69 (PB10)
- net BCK SPEAKER: now also VQ1.41 (PA5)
- net BCK STEREO OUT: now also VQ1.133 (PB3)
- net Chord A: now also VQ1.7 (PC13)
- net Chord Ab: now also VQ1.28 (PC2_C)
- net Chord B: now also VQ1.13 (PF3)
- net Chord Bb: now also VQ1.12 (PF2)
- net Chord C: now also VQ1.14 (PF4)
- net Chord D: now also VQ1.18 (PF6)
- net Chord Db: now also VQ1.15 (PF5)
- net Chord E: now also VQ1.20 (PF8)
- net Chord Eb: now also VQ1.19 (PF7)
- net Chord F: now also VQ1.21 (PF9)
- net Chord G: now also VQ1.26 (PC0)
- net Chord Gb: now also VQ1.22 (PF10)
- net DIN HEADPHONE: now also VQ1.27 (PC1)
- net DIN SPEAKER: now also VQ1.43 (PA7)
- net DIN STEREO OUT: now also VQ1.48 (PB2)
- net DN USB: now also U27.5
- net DP USB: now also U27.6
- net Extention: now also VQ1.42 (PA6)
- net GND: now also CN2.6, CN2.7, CN3.2, CN3.6, CN3.7, Card1.10, Card1.11, Card1.12, Card1.13, Card1.6 (VSS), FPC1.1, FPC1.10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
- net GPIO3 HEADPHONE: now also VQ1.49 (PF11)
- net GPIO3 SPEAKER: now also VQ1.57 (PG1)
- net GPIO3 STEREO OUT: now also VQ1.44 (PC4)
- net GPIO4 HEADPHONE: now also VQ1.50 (PF12)
- net GPIO4 SPEAKER: now also VQ1.64 (PE11)
- net GPIO4 STEREO OUT: now also VQ1.45 (PC5)
- net GPIO5 HEADPHONE: now also VQ1.53 (PF13)
- net GPIO5 SPEAKER: now also VQ1.65 (PE12)
- net GPIO5 STEREO OUT: now also VQ1.46 (PB0)
- net GPIO6 HEADPHONE: now also VQ1.56 (PG0)
- net GPIO6 SPEAKER: now also VQ1.66 (PE13)
- net GPIO6 STEREO OUT: now also VQ1.47 (PB1)
- net HEADPHONE GPIO L: now also VQ1.67 (PE14)
- net HEADPHONE GPIO R: now also VQ1.68 (PE15)
- net INT_N USB: now also U27.3
- net LRCK HEADPHONE: now also VQ1.73 (PB12)
- net LRCK SPEAKER: now also VQ1.110 (PA15)
- net LRCK STEREO OUT: now also VQ1.40 (PA4)
- net MUTE SUB: now also VQ1.140 (PB9)
- net MUTE TWEET/WOOF: now also VQ1.142 (PE1)
- net Mayor: now also VQ1.29 (PC3_C)
- net Minor: now also VQ1.36 (PA2)
- net SCL USB: now also U27.2; no longer R2.1, U32.B3 (SCL)
- net SDA USB: now also U27.1; no longer R1.2, U32.C3 (SDA)
- net SS XRES GPIO: now also VQ1.76 (PB15)
- net STEREO GPIO L/MONO: now also VQ1.134 (PB4)
- net STEREO GPIO R: now also VQ1.135 (PB5)
- net SUB AMP N: now also J10.2 (Pin_2)
- net SUB AMP P: now also J10.1 (Pin_1)
- net SYS: no longer C62.1, C63.1, U35.2 (VIN), U35.3 (EN)
- net TWEET AMP N: now also J8.2 (Pin_2)
- net TWEET AMP P: now also J8.1 (Pin_1)
- net VBUS: now also C62.1, C63.1, U35.2 (VIN), U35.3 (EN)
- net WOOF AMP N: now also J9.2 (Pin_2)
- net WOOF AMP P: now also J9.1 (Pin_1)
- net /SD SUB: now also VQ1.141 (PE0)
- net /SD TWEET/WOOF: now also VQ1.143 (PDR_ON)
- net Touch Pad Volume Encoder A: now reaches SW52.A
- net Touch Pad Volume Encoder A: now also VQ1.125 (PG10)
- net Touch Pad Volume Encoder B: now reaches SW52.B
- net Touch Pad Volume Encoder B: now also VQ1.124 (PG9)
- net PEDAL GPIO: now reaches J5.6
- net PEDAL GPIO: now also VQ1.77 (PD8), R127.2
- net Octave Down Switch: now reaches SW58.1
- net Octave Down Switch: now also SW58.2, VQ1.89 (PG4)
- net Keyboard Volume Encoder A: now reaches SW54.A
- net Keyboard Volume Encoder A: now also VQ1.129 (PG14)
- net Keyboard Volume Encoder B: now reaches SW54.B
- net Keyboard Volume Encoder B: now also VQ1.128 (PG13)
- net Recording Mode Switch: now reaches U11.4
- net Recording Mode Switch: now also U11.5, U11.6, VQ1.91 (PG6)
- net Chords Volume Encoder A: now reaches SW51.A
- net Chords Volume Encoder A: now also VQ1.127 (PG12)
- net Chords Volume Encoder B: now reaches SW51.B
- net Chords Volume Encoder B: now also VQ1.126 (PG11)
- net at CN2.4: now also R123.2
- net at CN2.5: now also D26.2 (A), OC1.2
- net Rythm Volume Encoder A: now reaches SW53.A
- net Rythm Volume Encoder A: now also VQ1.117 (PD3)
- net Rythm Volume Encoder B: now reaches SW53.B
- net Rythm Volume Encoder B: now also VQ1.109 (PA14)
- net LCD SCL: now reaches VQ1.1 (PE2)
- net LCD SCL: now also FPC1.4
- net SDA I2C2: now reaches VQ1.10 (PF0)
- net at VQ1.101 (PA9): now also R120.1, R121.2
- net INT_N USB 2: now reaches VQ1.102 (PA10)
- net INT_N USB 2: now also U36.3
- net DN USB 2: now reaches VQ1.103 (PA11)
- net DN USB 2: now also U36.5
- net DP USB 2: now reaches VQ1.104 (PA12)
- net DP USB 2: now also U36.6
- net at VQ1.106 (VCAP): now also VQ1.71 (VCAP), C208.1, C209.1
- net SCL I2C2: now reaches VQ1.11 (PF1)
- net SD D2: now reaches VQ1.111 (PC10)
- net SD D2: now also Card1.1 (DAT2), R115.1
- net SD D3: now reaches VQ1.112 (PC11)
- net SD D3: now also Card1.2 (CD/DAT3), R114.1
- net SD CLX: now reaches VQ1.113 (PC12)
- net SD CLX: now also Card1.5 (CLX)
- net IO2: now reaches VQ1.114 (PD0)
- net IO2: now also R108.2
- net IO3: now reaches VQ1.115 (PD1)
- net IO3: now also R107.2
- net SD CMD: now reaches VQ1.116 (PD2)
- net SD CMD: now also Card1.3 (CMD), R113.1
- net #RE: now reaches VQ1.118 (PD4)
- net #RE: now also U6.8
- net #WE: now reaches VQ1.119 (PD5)
- net #WE: now also U6.18
- net Vibrato Encoder B: now reaches VQ1.122 (PD6)
- net Vibrato Encoder B: now also SW55.B
- net Vibrato Encoder A: now reaches VQ1.123 (PD7)
- net Vibrato Encoder A: now also SW55.A
- net Main Volume Encoder B: now reaches VQ1.132 (PG15)
- net Main Volume Encoder B: now also SW50.B
- net SCL I2C1: now reaches VQ1.136 (PB6)
- net SCL I2C1: now also R2.1, U32.B3 (SCL), U36.2
- net SDA I2C1: now reaches VQ1.137 (PB7)
- net SDA I2C1: now also R1.2, U32.C3 (SDA), U36.1
- net at VQ1.138 (BOOT0): now also R119.2, SW59.1
- net Main Volume Encoder A: now reaches VQ1.139 (PB8)
- net Main Volume Encoder A: now also SW50.A
- net LCD RESET: now reaches VQ1.2 (PE3)
- net LCD RESET: now also FPC1.6
- net at VQ1.23 (PH0-OSC_IN): now also C214.2, U37.3
- net at VQ1.24 (PH1-OSC_OUT): now also C213.2, U37.1
- net at VQ1.25 (NRST): now also R126.2, SW60.1
- net LCD CS: now reaches VQ1.3 (PE4)
- net LCD CS: now also FPC1.2
- net TX MIDI: now reaches VQ1.34 (PA0)
- net TX MIDI: now also R125.1
- net LCD RS: now reaches VQ1.4 (PE5)
- net LCD RS: now also FPC1.3
- net LCD SDA: now reaches VQ1.5 (PE6)
- net LCD SDA: now also FPC1.5
- net SCL I2C4: now reaches VQ1.54 (PF14)
- new net: R122.2, U6.19
- new net: R109.1, U6.30
- new net: R56.1, U6.43
- new net: R110.1, U6.29
- new net: R108.1, U6.31
- new net: R107.1, U6.32
- new net: R106.1, U6.41
- new net: R57.1, U6.42
- new net: R55.1, U6.44
- new net: D26.1 (K), OC1.1, R123.1
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Other:
- note added: "Advanced Functionalities"
- note removed: "Advanced Funtionalities"
- note removed: "DIN-MIDI"
- note removed: "External Micro SD Card"
- note removed: "Midi"
- note removed: "USB-MIDI"
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