File: hardware/om-god.kicad_sch (KiCad schematic)
At the start: 530 parts, among them CN2 DIN-504B-M10, CN3 DIN-504B-M10, J1 Conn_01x13_Pin, J10 Conn_01x02_Socket, J11 Conn_01x08_Pin, J2 Conn_01x03_Pin, J3 PJ-625G, J4 PJ-625G, J5 PJ-625G, J6 Conn_01x08_Pin, J8 Conn_01x02_Socket, J9 Conn_01x02_Socket, Q1 Si7617DN, Q2 Si7617DN, Q3 Si7617DN, SW1 TS-1003ST-26, SW10 TS-1003ST-26, SW11 TS-1003ST-26, SW12 TS-1003ST-26, SW13 TS-1003ST-26, SW14 TS-1003ST-26, SW15 TS-1003ST-26, SW16 TS-1003ST-26, SW17 TS-1003ST-26, SW18 TS-1003ST-26, SW19 TS-1003ST-26, SW2 TS-1003ST-26, SW20 TS-1003ST-26, SW21 TS-1003ST-26, SW22 TS-1003ST-26, SW23 TS-1003ST-26, SW24 TS-1003ST-26, SW25 TS-1003ST-26, SW26 TS-1003ST-26, SW27 TS-1003ST-26, SW28 TS-1003ST-26, SW29 TS-1003ST-26, SW3 TS-1003ST-26, SW30 TS-1003ST-26, SW31 TS-1003ST-26, SW32 TS-1003ST-26, SW33 TS-1003ST-26, SW34 TS-1003ST-26, SW35 TS-1003ST-26, SW36 TS-1003ST-26, SW37 TS-1003ST-26, SW38 TS-1003ST-26, SW39 TS-1003ST-26, SW4 TS-1003ST-26, SW40 TS-1003ST-26, SW41 TS-1003ST-26, SW42 TS-1003ST-26, SW43 TS-1003ST-26, SW44 TS-1003ST-26, SW45 TS-1003ST-26, SW46 TS-1003ST-26, SW47 TS-1003ST-26, SW48 TS-1003ST-26, SW49 RotaryEncoder_Switch, SW5 TS-1003ST-26, SW50 RotaryEncoder, SW51 RotaryEncoder, SW52 RotaryEncoder, SW53 RotaryEncoder, SW54 RotaryEncoder, SW55 RotaryEncoder, SW56 TS-1003ST-26, SW57 TS-1003ST-26, SW58 TS-1003ST-26, SW59 SW_Push, SW6 TS-1003ST-26, SW60 SW_Push, SW7 TS-1003ST-26, SW8 TS-1003ST-26, SW9 TS-1003ST-26, U1 NE5532DR, U12 LMR33630ADDAR, U13 LMR33630ADDAR, U14 LMR33630ADDAR, U15 TPS54202DDC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

Commit message: h
Parts:
- removed C211: 100nF, Capacitor_SMD:C_0402_1005Metric, symbol Device:C
- removed D32: SB520, PCM_Diode_THT_AKL:D_DO-201AD_P12.70mm_Horizontal, symbol PCM_Diode_Schottky_AKL:SB520
- removed R33, R34, R37, R40: 100K, Resistor_SMD:R_0402_1005Metric, symbol Device:R
- removed R61: 6K, Resistor_SMD:R_0402_1005Metric, symbol Device:R
- removed SW11, SW12: TS-1003ST-26, lcsc:SW-SMD_4P-L12.0-W12.0-P5.00-LS15.4, symbol lcsc:TS-1003ST-26
- added C179, C184: 10uF, Capacitor_SMD:C_0603_1608Metric, symbol Device:C
- added C185: 220nF, Capacitor_SMD:C_0402_1005Metric, symbol Device:C
- added C191, C193, C197: 1uF, Capacitor_SMD:C_0402_1005Metric, symbol Device:C
- added C192: 220nF, Capacitor_SMD:C_0603_1608Metric, symbol Device:C
- added C201: 0.1uF, Capacitor_SMD:C_0402_1005Metric, symbol Device:C
- added C207: 47pF, Capacitor_SMD:C_0603_1608Metric, symbol Device:C
- added C210: 47pF, Capacitor_SMD:C_0402_1005Metric, symbol Device:C
- added C213, C218, C219, C224, C225, C230, C231, C234: 22uF, Capacitor_SMD:C_0603_1608Metric, symbol Device:C
- added D49: LED, lcsc:LED0603-RD, symbol Device:LED
- added J11: Conn_01x02_Socket, lcsc:CONN-TH_2P-P5.00_WJ500V-5.08-2P, symbol Connector:Conn_01x02_Socket
- added L13: 15uH, lcsc:IND-SMD_L12.3-W12.3, symbol Device:L
- added L15: 6.8uH, lcsc:IND-SMD_L3.2-W2.5_L3225, symbol Device:L
- added R115, R116: 10K, Resistor_SMD:R_0402_1005Metric, symbol Device:R
- added R117, R54: 1K, Resistor_SMD:R_0402_1005Metric, symbol Device:R
- added R125, R131: 100K, Resistor_SMD:R_0402_1005Metric, symbol Device:R
- added R126: 9.09K, Resistor_SMD:R_0402_1005Metric, symbol Device:R
- added R132: 43.2K, Resistor_SMD:R_0402_1005Metric, symbol Device:R
- added R18: 5K, Resistor_SMD:R_0402_1005Metric, symbol Device:R
- added R35: 470, Resistor_SMD:R_0402_1005Metric, symbol Device:R
- added SW47, SW51: TS-1003ST-26, lcsc:SW-SMD_4P-L12.0-W12.0-P5.00-LS15.4, symbol lcsc:TS-1003ST-26
- added U36, U39: LMR33630ADDAR, lcsc:ESOP-8_L4.9-W3.9-P1.27-LS6.0-TL-EP, symbol lcsc:LMR33630ADDAR
- C105: renamed from C118; footprint Capacitor_SMD:C_0402_1005Metric -> Capacitor_SMD:C_0603_1608Metric
- C106: renamed from C119; footprint Capacitor_SMD:C_0402_1005Metric -> Capacitor_SMD:C_0603_1608Metric
- C107: renamed from C125; footprint Capacitor_SMD:C_0402_1005Metric -> Capacitor_SMD:C_0603_1608Metric
- C108: renamed from C126; footprint Capacitor_SMD:C_0402_1005Metric -> Capacitor_SMD:C_0603_1608Metric
- C109: renamed from C33; footprint Capacitor_SMD:C_0402_1005Metric -> Capacitor_SMD:C_0603_1608Metric
- C110: renamed from C32; footprint Capacitor_SMD:C_0402_1005Metric -> Capacitor_SMD:C_0603_1608Metric
- C111: renamed from C120; footprint Capacitor_SMD:C_0402_1005Metric -> Capacitor_SMD:C_0603_1608Metric
- C112: renamed from C121; footprint Capacitor_SMD:C_0402_1005Metric -> Capacitor_SMD:C_0603_1608Metric
- C113: renamed from C127; footprint Capacitor_SMD:C_0402_1005Metric -> Capacitor_SMD:C_0603_1608Metric
- C114: renamed from C128; footprint Capacitor_SMD:C_0402_1005Metric -> Capacitor_SMD:C_0603_1608Metric
- C115: renamed from C34; footprint Capacitor_SMD:C_0402_1005Metric -> Capacitor_SMD:C_0603_1608Metric
- C116: renamed from C35; footprint Capacitor_SMD:C_0402_1005Metric -> Capacitor_SMD:C_0603_1608Metric
- C117: renamed from C6; footprint Capacitor_SMD:C_0402_1005Metric -> Capacitor_SMD:C_0603_1608Metric
- C118: renamed from C122; footprint Capacitor_SMD:C_0402_1005Metric -> Capacitor_SMD:C_0603_1608Metric
- C119: renamed from C123; footprint Capacitor_SMD:C_0402_1005Metric -> Capacitor_SMD:C_0603_1608Metric
- C120: renamed from C129; footprint Capacitor_SMD:C_0402_1005Metric -> Capacitor_SMD:C_0603_1608Metric
- C121: renamed from C130; footprint Capacitor_SMD:C_0402_1005Metric -> Capacitor_SMD:C_0603_1608Metric
- C122: renamed from C36; footprint Capacitor_SMD:C_0402_1005Metric -> Capacitor_SMD:C_0603_1608Metric
- C123: renamed from C37; footprint Capacitor_SMD:C_0402_1005Metric -> Capacitor_SMD:C_0603_1608Metric
- C165: renamed from C102; value 100nF -> 1uF
- C187: renamed from C165; footprint Capacitor_SMD:C_0603_1608Metric -> Capacitor_SMD:C_0402_1005Metric
- C19: renamed from C13; footprint Capacitor_THT:CP_Radial_D8.0mm_P3.50mm -> lcsc:CAP-SMD_BD4.0-L4.3-W4.3-FD
- C20: renamed from C14; footprint Capacitor_THT:CP_Radial_D8.0mm_P3.50mm -> lcsc:CAP-SMD_BD4.0-L4.3-W4.3-FD
- C206: value 4.7uF -> 0.1uF
- C209: renamed from C168; footprint Capacitor_SMD:C_0402_1005Metric -> Capacitor_SMD:C_0603_1608Metric
- C21: renamed from C15; footprint Capacitor_THT:CP_Radial_D8.0mm_P3.50mm -> lcsc:CAP-SMD_BD4.0-L4.3-W4.3-FD
- C22: renamed from C16; footprint Capacitor_THT:CP_Radial_D8.0mm_P3.50mm -> lcsc:CAP-SMD_BD4.0-L4.3-W4.3-FD
- C220: renamed from C71; footprint Capacitor_SMD:C_0402_1005Metric -> Capacitor_SMD:C_0603_1608Metric
- C226: renamed from C173; footprint Capacitor_SMD:C_0402_1005Metric -> Capacitor_SMD:C_0603_1608Metric
- C23: renamed from C17; footprint Capacitor_THT:CP_Radial_D8.0mm_P3.50mm -> lcsc:CAP-SMD_BD4.0-L4.3-W4.3-FD
- C232: renamed from C174; footprint Capacitor_SMD:C_0402_1005Metric -> Capacitor_SMD:C_0603_1608Metric
- C24: renamed from C193; footprint Capacitor_THT:CP_Radial_D8.0mm_P3.50mm -> lcsc:CAP-SMD_BD4.0-L4.3-W4.3-FD
- C25: renamed from C192; footprint Capacitor_THT:CP_Radial_D8.0mm_P3.50mm -> lcsc:CAP-SMD_BD4.0-L4.3-W4.3-FD
- C26: renamed from C184; footprint Capacitor_THT:CP_Radial_D8.0mm_P3.50mm -> lcsc:CAP-SMD_BD4.0-L4.3-W4.3-FD
- C27: renamed from C187; footprint Capacitor_THT:CP_Radial_D8.0mm_P3.50mm -> lcsc:CAP-SMD_BD4.0-L4.3-W4.3-FD
- C28: renamed from C190; footprint Capacitor_THT:CP_Radial_D8.0mm_P3.50mm -> lcsc:CAP-SMD_BD4.0-L4.3-W4.3-FD
- C29: renamed from C87; footprint Capacitor_THT:CP_Radial_D8.0mm_P3.50mm -> lcsc:CAP-SMD_BD4.0-L4.3-W4.3-FD
- C30: renamed from C88; footprint Capacitor_THT:CP_Radial_D8.0mm_P3.50mm -> lcsc:CAP-SMD_BD4.0-L4.3-W4.3-FD
- C31: renamed from C89; footprint Capacitor_THT:CP_Radial_D8.0mm_P3.50mm -> lcsc:CAP-SMD_BD4.0-L4.3-W4.3-FD
- C32: renamed from C90; footprint Capacitor_THT:CP_Radial_D8.0mm_P3.50mm -> lcsc:CAP-SMD_BD4.0-L4.3-W4.3-FD
- C33: renamed from C91; footprint Capacitor_THT:CP_Radial_D8.0mm_P3.50mm -> lcsc:CAP-SMD_BD4.0-L4.3-W4.3-FD
- renumbered C2 to C1, C185 to C10, C26 to C100, C116 to C101, C40 to C102, C117 to C103, C27 to C104, C186 to C11, C188 to C12, C7 to C124, C144 to C125, C142 to C126, C146 to C127, C140 to C128, C175 to C129, C189 to C13, C145 to C130, C141 to C131, C176 to C132, C177 to C133, C99 to C134, C151 to C136, C178 to C137, C157 to C138, C179 to C139, C82 to C14, C210 to C140, C139 to C141, C137 to C142, C147 to C143, C207 to C144, C1 to C145, C203 to C146, C180 to C147, C149 to C148, C138 to C149, C83 to C15, C100 to C150, C204 to C151, C143 to C152, C181 to C153, C182 to C154, C205 to C155, C183 to C157, C155 to C158, C202 to C159, C84 to C16, C152 to C160, C201 to C161, C153 to C162, C148 to C163, C200 to C164, C199 to C166, C150 to C167, C215 to C168, C216 to C169, C85 to C17, C214 to C170, C213 to C171, C101 to C172, C154 to C173, C198 to C174, C197 to C175, C63 to C176, C64 to C177, C103 to C178, C86 to C18, C44 to C180, C164 to C181, C62 to C182, C65 to C183, C45 to C186, C208 to C188, C61 to C189, C66 to C190, C67 to C194, C166 to C195, C209 to C196, C98 to C198, C55 to C199, C191 to C2, C158 to C200, C68 to C202, C167 to C203, C56 to C204, C159 to C205, C69 to C208, C57 to C211, C160 to C212, C70 to C214, C169 to C215, C58 to C216, C161 to C217, C170 to C221, C59 to C222, C162 to C223, C171 to C227, C60 to C228, C163 to C229, C172 to C233, C81 to C3, C18 to C34, C80 to C35, C196 to C36, C195 to C37, C92 to C38, C93 to C39, C3 to C4, C46 to C40, C43 to C41, C8 to C42, C19 to C43, C47 to C44, C20 to C45, C77 to C46, C75 to C47, C78 to C48, C79 to C49, C9 to C5, C53 to C50, C41 to C51, C54 to C52, C48 to C53, C42 to C54, C104 to C55, C72 to C56, C73 to C57, C212 to C58, C51 to C59, C10 to C6, C49 to C60, C134 to C61, C133 to C62, C52 to C63, C76 to C64, C74 to C65, C50 to C66, C22 to C67, C105 to C68, C106 to C69, C11 to C7, C107 to C70, C124 to C71, C24 to C72, C23 to C73, C132 to C74, C136 to C75, C135 to C76, C21 to C77, C131 to C78, C4 to C79, C12 to C8, C94 to C80, C97 to C81, C95 to C82, C96 to C83, C5 to C84, C108 to C85, C38 to C86, C109 to C87, C25 to C88, C110 to C89, C194 to C9, C111 to C90, C112 to C91, C113 to C92, C28 to C93, C29 to C94, C31 to C95, C30 to C96, C114 to C97, C39 to C98, C115 to C99, CN2 to CN1, CN3 to CN2, D63 to D10, D6 to D11, D7 to D12, D52 to D13, D64 to D14, D8 to D15, D9 to D16, D53 to D17, D65 to D18, D10 to D19, D61 to D2, D11 to D20, D54 to D21, D66 to D22, D12 to D23, D13 to D24, D55 to D25, D67 to D26, D14 to D27, D15 to D28, D56 to D29, D2 to D3, D68 to D30, D16 to D31, D17 to D32, D57 to D33, D69 to D34, D18 to D35, D19 to D36, D58 to D37, D70 to D38, D20 to D39, D3 to D4, D21 to D40, D59 to D41, D71 to D42, D22 to D43, D23 to D44, D60 to D45, D72 to D46, D24 to D47, D25 to D48, D50 to D5, D26 to D50, D27 to D51, D29 to D52, D30 to D53, D31 to D54, D28 to D55, D62 to D6, D4 to D7, D5 to D8, D51 to D9, J3 to J1, J11 to J10, J4 to J2, J1 to J3, J2 to J4, J9 to J7, J10 to J9, L3 to L1, L4 to L10, L13 to L11, L14 to L12, L5 to L14, L7 to L2, L10 to L3, L11 to L4, L1 to L5, L2 to L6, L6 to L7, L12 to L9, R3 to R1, R65 to R10, R107 to R100, R108 to R101, R109 to R102, R110 to R103, R1 to R104, R96 to R105, R43 to R106, R44 to R107, R45 to R108, R126 to R109, R67 to R11, R95 to R110, R97 to R111, R98 to R112, R118 to R113, R117 to R114, R51 to R12, R31 to R121, R32 to R122, R35 to R123, R36 to R124, R41 to R127, R42 to R128, R38 to R129, R52 to R13, R39 to R130, R119 to R133, R120 to R134, R121 to R135, R30 to R14, R53 to R15, R7 to R16, R8 to R17, R72 to R19, R4 to R2, R73 to R20, R27 to R21, R82 to R22, R83 to R23, R75 to R24, R28 to R25, R124 to R26, R123 to R27, R125 to R28, R84 to R29, R47 to R3, R50 to R30, R76 to R31, R78 to R32, R85 to R33, R29 to R34, R77 to R36, R81 to R37, R79 to R38, R80 to R39, R46 to R4, R9 to R40, R16 to R41, R12 to R42, R11 to R43, R18 to R44, R17 to R45, R13 to R46, R62 to R47, R63 to R48, R10 to R49, R48 to R5, R26 to R50, R23 to R51, R127 to R52, R60 to R53, R6 to R55, R59 to R56, R5 to R57, R115 to R58, R114 to R59, R49 to R6, R113 to R60, R112 to R61, R111 to R62, R116 to R63, R19 to R64, R20 to R65, R24 to R66, R25 to R67, R14 to R68, R15 to R69, R21 to R7, R68 to R70, R70 to R71, R71 to R72, R92 to R73, R90 to R74, R74 to R75, R88 to R76, R89 to R77, R69 to R78, R87 to R79, R22 to R8, R66 to R80, R86 to R81, R93 to R82, R122 to R83, R91 to R84, R58 to R85, R2 to R86, R54 to R87, R104 to R88, R102 to R89, R64 to R9, R103 to R90, R105 to R91, R99 to R92, R100 to R93, R101 to R94, R94 to R95, R55 to R96, R56 to R97, R57 to R98, R106 to R99, SW53 to SW10, SW3 to SW11, SW15 to SW12, SW27 to SW13, SW39 to SW14, SW4 to SW15, SW28 to SW17, SW40 to SW18, SW51 to SW19, SW13 to SW2, SW52 to SW20, SW5 to SW21, SW17 to SW22, SW29 to SW23, SW41 to SW24, SW6 to SW25, SW18 to SW26, SW30 to SW27, SW42 to SW28, SW7 to SW29, SW25 to SW3, SW19 to SW30, SW43 to SW32, SW54 to SW33, SW55 to SW34, SW8 to SW35, SW20 to SW36, SW32 to SW37, SW44 to SW38, SW9 to SW39, SW37 to SW4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
Connections:
- net +12V: now also C207.1, C213.1, C219.1, C225.1, C231.1, L13.2, R125.2
- net +3.3V: now also VQ1.95 (VDD33USB), R18.2, R35.2; no longer C206.1, OC1.4, VQ1.35 (PA1), VQ1.6 (VBAT)
- net +BATT: now also C184.1, C192.1, J11.1 (Pin_1), U39.2 (VIN), U39.3 (EN)
- net Chord A: now also SW2.3, SW2.4, SW3.3, SW3.4, SW4.3, SW4.4; no longer SW52.3, SW52.4, SW8.3, SW8.4
- net Chord Ab: now also SW52.3, SW52.4, SW53.3, SW53.4, SW51.3, SW51.4; no longer SW43.3, SW43.4, SW48.3, SW48.4, SW50.3, SW50.4
- net Chord B: now also SW11.3, SW11.4, SW12.3, SW12.4, SW13.3, SW13.4, SW14.3, SW14.4; no longer SW23.3, SW23.4, SW27.3, SW27.4, SW3.3, SW3.4, SW7.3, SW7.4
- net Chord Bb: now also SW6.3, SW6.4, SW7.3, SW7.4, SW8.3, SW8.4, SW9.3, SW9.4; no longer SW13.3, SW13.4, SW17.3, SW17.4, SW2.3, SW2.4
- net Chord C: now also SW15.3, SW15.4, SW16.3, SW16.4, SW17.3, SW17.4, SW18.3, SW18.4; no longer SW12.3, SW12.4, SW31.3, SW31.4, SW37.3, SW37.4, SW6.3, SW6.4
- net Chord D: now also SW25.3, SW25.4, SW26.3, SW26.4, SW27.3, SW27.4, SW28.3, SW28.4; no longer SW15.3, SW15.4, SW22.3, SW22.4, SW49.3, SW49.4, SW53.3, SW53.4
- net Chord Db: now also SW21.3, SW21.4, SW22.3, SW22.4, SW23.3, SW23.4, SW24.3, SW24.4; no longer SW11.3, SW11.4, SW16.3, SW16.4, SW41.3, SW41.4, SW45.3, SW45.4
- net Chord E: now also SW35.3, SW35.4, SW36.3, SW36.4, SW37.3, SW37.4, SW38.3, SW38.4; no longer SW14.3, SW14.4, SW18.3, SW18.4, SW25.3, SW25.4, SW30.3, SW30.4
- net Chord Eb: now also SW29.3, SW29.4, SW30.3, SW30.4, SW31.3, SW31.4, SW32.3, SW32.4; no longer SW21.3, SW21.4, SW26.3, SW26.4, SW4.3, SW4.4, SW9.3, SW9.4
- net Chord F: now also SW39.3, SW39.4, SW40.3, SW40.4, SW41.3, SW41.4, SW42.3, SW42.4; no longer SW24.3, SW24.4, SW28.3, SW28.4, SW29.3, SW29.4, SW36.3, SW36.4
- net Chord G: now also SW48.3, SW48.4, SW49.3, SW49.4, SW50.3, SW50.4, SW47.3, SW47.4; no longer SW39.3, SW39.4, SW42.3, SW42.4, SW44.3, SW44.4, SW46.3, SW46.4
- net Chord Gb: now also SW43.3, SW43.4, SW44.3, SW44.4, SW45.3, SW45.4, SW46.3, SW46.4; no longer SW32.3, SW32.4, SW35.3, SW35.4, SW38.3, SW38.4, SW40.3, SW40.4
- net GND: now also U12.5, U17.21 (EP), U21.25 (EP), C179.2, C184.2, C185.2, C191.1, C192.2, C193.2, C197.2, C213.2, C218.2, C219.2, C224.2, C225.2, C230.2, C231.2, C234.2, D49.1 (K), J11.2 (Pin_2), R126.1, R132.1, U36.1 (PGND), U36.9 (EP), U39.1 (PGND), U39.9 (EP); no longer C206.2, J10.8 (Pin_8), J6.8 (Pin_8), U10.6, U12.1, U12.2, U12.3, U13.2, U14.2, U9.6, VQ1.100 (PA8), VQ1.105 (PA13), VQ1.92 (PG7), VQ1.93 (PG8), VQ1.95 (VDD33USB)
- net HEADPHONE AMP L: now also R117.2
- net HEADPHONE AMP R: now also R54.1
- net MONO BUFF: now also R116.1; no longer R16.2, R17.1, U8.7 (IN1-)
- net Recording Mode Switch: no longer U12.4, U12.5
- net SPEAKER SUM BUFF: now also R115.1; no longer R7.2, R8.1, U4.7 (IN1-)
- net SYS: now also C179.1, C185.1, U36.2 (VIN), U36.3 (EN)
- net TWEET AMP N: now also J8.1 (Pin_1); no longer J8.2 (Pin_2)
- net TWEET AMP P: now also J8.2 (Pin_2); no longer J8.1 (Pin_1)
- net at R39.1, U17.16 (RIN-): now also R54.2
- net at R32.1, U17.5 (LIN-): now also R117.1
- net at SW48.1, SW48.2: now also D42.2 (A); no longer D46.2 (A)
- net at SW6.1, SW6.2: now also D5.2 (A); no longer D13.2 (A)
- net at SW40.1, SW40.2: now also D34.2 (A); no longer D38.2 (A)
- net at SW38.1, SW38.2: now also D32.2 (A); no longer D40.2 (A)
- net at SW8.1, SW8.2: now also D7.2 (A); no longer D4.2 (A)
- net at SW43.1, SW43.2: now also D37.2 (A); no longer D45.2 (A)
- net at SW16.1, SW16.2: now also D14.2 (A); no longer D18.2 (A)
- net at SW52.1, SW52.2: now also D46.2 (A); no longer D3.2 (A)
- net at SW28.1, SW28.2: now also D24.2 (A); no longer D36.2 (A)
- net at SW29.1, SW29.2: now also D25.2 (A); no longer D33.2 (A)
- net at SW50.1, SW50.2: now also D44.2 (A); no longer D47.2 (A)
- net at SW7.1, SW7.2: now also D6.2 (A); no longer D10.2 (A)
- net at SW17.1, SW17.2: now also D15.2 (A); no longer D8.2 (A)
- net at D2.2 (A): now also SW2.1, SW2.2
- net at SW37.1, SW37.2: now also D31.2 (A); no longer D16.2 (A)
- net at SW25.1, SW25.2: now also D21.2 (A); no longer D29.2 (A)
- net at SW12.1, SW12.2: now also D10.2 (A); no longer D14.2 (A)
- net at SW49.1, SW49.2: now also D43.2 (A); no longer D23.2 (A)
- net at SW32.1, SW32.2: now also D28.2 (A); no longer D39.2 (A)
- net at SW18.1, SW18.2: now also D16.2 (A); no longer D32.2 (A)
- net at SW53.1, SW53.2: now also D47.2 (A); no longer D24.2 (A)
- net at SW21.1, SW21.2: now also D17.2 (A); no longer D25.2 (A)
- net at SW3.1, SW3.2: now also D3.2 (A); no longer D9.2 (A)
- net at SW14.1, SW14.2: now also D12.2 (A); no longer D31.2 (A)
- net at SW46.1, SW46.2: now also D40.2 (A); no longer D44.2 (A)
- net at SW27.1, SW27.2: now also D23.2 (A); no longer D12.2 (A)
- net at SW45.1, SW45.2: now also D39.2 (A); no longer D20.2 (A)
- net at SW30.1, SW30.2: now also D26.2 (A); no longer D30.2 (A)
- net at SW4.1, SW4.2: now also D4.2 (A); no longer D27.2 (A)
- net at SW9.1, SW9.2: now also D8.2 (A); no longer D28.2 (A)
- net at SW31.1, SW31.2: now also D27.2 (A); no longer D15.2 (A)
- net at SW15.1, SW15.2: now also D13.2 (A); no longer D21.2 (A)
- net at SW11.1, SW11.2: now also D9.2 (A); no longer D17.2 (A)
- net at SW22.1, SW22.2: now also D18.2 (A); no longer D22.2 (A)
- net at SW24.1, SW24.2: now also D20.2 (A); no longer D35.2 (A)
- net at SW42.1, SW42.2: now also D36.2 (A); no longer D43.2 (A)
- net at SW26.1, SW26.2: now also D22.2 (A); no longer D26.2 (A)
- net at SW39.1, SW39.2: now also D33.2 (A); no longer D41.2 (A)
- net at SW41.1, SW41.2: now also D35.2 (A); no longer D19.2 (A)
- net at SW35.1, SW35.2: now also D29.2 (A); no longer D37.2 (A)
- net at U9.2: now also D49.2 (A)
- net at U9.3: now also R18.1
- net at SW23.1, SW23.2: now also D19.2 (A); no longer D11.2 (A)
- net at SW44.1, SW44.2: now also D38.2 (A); no longer D42.2 (A)
- net at SW36.1, SW36.2: now also D30.2 (A); no longer D34.2 (A)
- net at SW13.1, SW13.2: now also D11.2 (A); no longer D7.2 (A)
- removed net PG: U34.4 (PG), U35.4 (PG), U37.4 (PG), U38.4 (PG)
- new net: D45.2 (A), SW51.1, SW51.2
- new net: C210.2, R131.1, R132.2, U39.5 (FB)
- new net: R115.2, R7.2, R8.1, U4.7 (IN1-)
- new net: C206.1, L15.1, U39.8 (SW)
- new net: C206.2, U39.7 (BOOT)
- new net: C197.1, U39.6 (VCC)
- new net: C201.1, L13.1, U36.8 (SW)
- new net: R116.2, R16.2, R17.1, U8.7 (IN1-)
- new net: C201.2, U36.7 (BOOT)
- new net: C193.1, U36.6 (VCC)
- new net: C207.2, R125.1, R126.2, U36.5 (FB)
- new net: D41.2 (A), SW47.1, SW47.2
- new net 3.3BATT: C191.2, C210.1, C218.1, C224.1, C230.1, C234.1, J10.8 (Pin_8), J6.8 (Pin_8), L15.2, R131.2, VQ1.6 (VBAT)
- new net Main On/Off Switch: U9.6, VQ1.105 (PA13)
- new net Metronome On/Off Switch: U14.2, VQ1.100 (PA8)
- new net RX MIDI: OC1.4, R35.1, VQ1.35 (PA1)
- new net Rythm On/Off Switch: U13.2, VQ1.93 (PG8)
- new net Sustain On/Off Switch: U10.6, VQ1.92 (PG7)
- no-connect marks 81 -> 89
Other:
- moved on the sheet: C129, C132, C133, C137, C139, C147, C153, C154, C157, L7, R106, R107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

Commit message: j
Parts:
- removed R113, R114: 0, Resistor_SMD:R_0402_1005Metric, symbol Device:R
- added FB1: 100, Inductor_SMD:L_0603_1608Metric, symbol Device:FerriteBead
- C117: footprint Capacitor_SMD:C_0603_1608Metric -> Capacitor_SMD:C_0402_1005Metric
- C173: footprint Capacitor_SMD:C_0402_1005Metric -> Capacitor_SMD:C_0603_1608Metric
- C46, C47, C48, C49, C64, C65: footprint PCM_Capacitor_THT_AKL:C_Rect_L4.0mm_W2.5mm_P2.50mm -> Capacitor_SMD:C_0603_1608Metric
Connections:
- net STEREO OUT DAC L is gone; now on net STEREO DAC L: C38.1, R5.2
- net STEREO OUT DAC R is gone; now on net STEREO DAC R: C39.1, R6.2
- net +3.3V: now also FB1.1
- net +3.3VA: now also FB1.2
- net MONO BUFF: now also U15.7 (NC2); no longer U15.9 (NC1)
- net STEREO BUFF L: now also U15.4 (NO2), U6.2 (OUT2), U6.3 (IN2-); no longer U15.2 (NO1), U6.7 (IN1-), U6.8 (OUT1)
- net STEREO BUFF L/MONO: now also U15.6 (COM2); no longer U15.10 (COM1)
- net STEREO BUFF R: now also U6.7 (IN1-), U6.8 (OUT1); no longer U6.2 (OUT2), U6.3 (IN2-)
- net STEREO DAC L: now also U6.4 (IN2+); no longer U6.6 (IN1+)
- net STEREO DAC R: now also U6.6 (IN1+); no longer U6.4 (IN2+)
- net STEREO/MONO GPIO: now also U15.5 (IN2); no longer U15.1 (IN1)
- net TWEET AMP N: now also C108.1, C114.1, L4.2, R67.2; no longer C106.1, C112.1, L2.2, R65.2
- net TWEET AMP P: now also C107.2, C113.2, L3.2, R66.1; no longer C105.2, C111.2, L1.2, R64.1
- net TWEET SUM BUFF: now also C70.2; no longer C68.2
- net TWEET SUM BUFF N: now also C71.2; no longer C69.2
- net WOOF AMP N: now also C106.1, C112.1, L2.2, R65.2; no longer C108.1, C114.1, L4.2, R67.2
- net WOOF AMP P: now also C105.2, C111.2, L1.2, R64.1; no longer C107.2, C113.2, L3.2, R66.1
- net WOOF SUM BUFF: now also C68.2; no longer C70.2
- net WOOF SUM BUFF N: now also C69.2; no longer C71.2
- net at C48.2, R13.1, R15.2: no longer C49.2, R15.1, U7.4 (IN2+)
- new net: C49.2, R15.1, U7.4 (IN2+)
- no-connect marks 89 -> 90
Other:
- moved on the sheet: C48, C60, J7, J8

Commit message: added stuff
Parts:
- removed R33: 10K, Resistor_SMD:R_0402_1005Metric, symbol Device:R
- removed SW59: RotaryEncoder_Switch, lcsc:SW-TH_EC11E1820402, symbol Device:RotaryEncoder_Switch
- added SW61: RotaryEncoder_Switch, lcsc:SW-TH_EC11E15244G1, symbol Device:RotaryEncoder_Switch
Connections:
- net +3.3V: now also J10.6 (Pin_6); no longer J6.5 (Pin_5)
- net +5V: now also J6.5 (Pin_5); no longer J10.6 (Pin_6)
- net Chords Volume Encoder A: now also VQ1.122 (PD6); no longer VQ1.127 (PG12)
- net Chords Volume Encoder B: now also VQ1.123 (PD7); no longer VQ1.126 (PG11)
- net Func Encoder A: now also SW61.A
- net Func Encoder B: now also SW61.B
- net Func Switch: now also SW61.D (S1)
- net GND: now also SW61.C, SW61.E (S2)
- net GPIO3 STEREO OUT: now also VQ1.46 (PB0); no longer VQ1.44 (PC4)
- net GPIO4 SPEAKER: now also VQ1.65 (PE12); no longer VQ1.64 (PE11)
- net GPIO4 STEREO OUT: now also VQ1.44 (PC4); no longer VQ1.45 (PC5)
- net GPIO5 SPEAKER: now also VQ1.64 (PE11); no longer VQ1.65 (PE12)
- net GPIO5 STEREO OUT: now also VQ1.45 (PC5); no longer VQ1.46 (PB0)
- net HEADPHONE GPIO L: now also VQ1.70 (PB11); no longer VQ1.67 (PE14)
- net IO4: now also VQ1.63 (PE10); no longer VQ1.58 (PE7)
- net IO5: now also VQ1.60 (PE9); no longer VQ1.59 (PE8)
- net IO6: now also VQ1.59 (PE8); no longer VQ1.60 (PE9)
- net IO7: now also VQ1.58 (PE7); no longer VQ1.63 (PE10)
- net IOFF 13: now also U21.18 (CS6); no longer U21.11 (CS13/GPO5)
- net IOFF 14: now also U21.19 (CS5); no longer U21.10 (CS14/GPO6)
- net IOFF 15: now also U21.20 (CS4); no longer U21.9 (CS15/SH/~{HI})
- net Keyboard Volume Encoder A: now also VQ1.128 (PG13); no longer VQ1.129 (PG14)
- net Keyboard Volume Encoder B: now also VQ1.129 (PG14); no longer VQ1.128 (PG13)
- net MUTE TWEET/WOOF: now also VQ1.78 (PD9); no longer VQ1.142 (PE1)
- net Main On/Off Switch: now also VQ1.93 (PG8); no longer VQ1.105 (PA13)
- net Main Volume Encoder A: now also VQ1.109 (PA14); no longer VQ1.139 (PB8)
- net Main Volume Encoder B: now also VQ1.117 (PD3); no longer VQ1.132 (PG15)
- net Rythm On/Off Switch: now also VQ1.97 (PC7); no longer VQ1.93 (PG8)
- net Rythm Volume Encoder A: now also VQ1.126 (PG11); no longer VQ1.117 (PD3)
- net Rythm Volume Encoder B: now also VQ1.127 (PG12); no longer VQ1.109 (PA14)
- net SCL I2C1: no longer R86.1, U29.B3 (SCL)
- net SCL USB: now also R86.1, U29.B3 (SCL)
- net SDA I2C1: no longer R104.2, U29.C3 (SDA)
- net SDA USB: now also R104.2, U29.C3 (SDA)
- net SS 10: now also U21.15 (CS9/GPO1); no longer U21.14 (CS10/GPO2)
- net SS 11: now also U21.16 (CS8/GPO0); no longer U21.13 (CS11/GPO3)
- net SS 12: now also U21.17 (CS7); no longer U21.12 (CS12/GPO4)
- net SS 4: now also U21.9 (CS15/SH/~{HI}); no longer U21.20 (CS4)
- net SS 5: now also U21.10 (CS14/GPO6); no longer U21.19 (CS5)
- net SS 6: now also U21.11 (CS13/GPO5); no longer U21.18 (CS6)
- net SS 7: now also U21.12 (CS12/GPO4); no longer U21.17 (CS7)
- net SS 8: now also U21.13 (CS11/GPO3); no longer U21.16 (CS8/GPO0)
- net SS 9: now also U21.14 (CS10/GPO2); no longer U21.15 (CS9/GPO1)
- net STEREO/MONO GPIO: now also VQ1.68 (PE15); no longer VQ1.78 (PD9)
- net TWEET AMP N: now also J8.2 (Pin_2); no longer J8.1 (Pin_1)
- net TWEET AMP P: now also J8.1 (Pin_1); no longer J8.2 (Pin_2)
- net Touch Pad Volume Encoder A: now also VQ1.124 (PG9); no longer VQ1.125 (PG10)
- net Touch Pad Volume Encoder B: now also VQ1.125 (PG10); no longer VQ1.124 (PG9)
- net Vibrato Encoder A: now also VQ1.132 (PG15); no longer VQ1.123 (PD7)
- net Vibrato Encoder B: now also VQ1.139 (PB8); no longer VQ1.122 (PD6)
- net WOOF AMP N: now also J7.1 (Pin_1); no longer J7.2 (Pin_2)
- net WOOF AMP P: now also J7.2 (Pin_2); no longer J7.1 (Pin_1)
- net /SD TWEET/WOOF: now also VQ1.67 (PE14); no longer VQ1.143 (PDR_ON)
- net DN USB renamed USB DN
- net DN USB 2 renamed USB 2 DN
- net DP USB renamed USB DP
- net DP USB 2 renamed USB 2 DP
- net HEADPHONE GPIO R: no longer names the net of AUDIO1.7
- net HEADPHONE GPIO R: no longer VQ1.68 (PE15)
- no-connect marks 90 -> 93

Commit message: d
Parts:
- removed C101, C103: 220uF, Capacitor_THT:CP_Radial_D8.0mm_P3.50mm, symbol Device:C_Polarized
- removed C105, C106, C107, C108: 680nF, Capacitor_SMD:C_0603_1608Metric, symbol Device:C
- removed C111, C112, C113, C114: 1uF, Capacitor_SMD:C_0603_1608Metric, symbol Device:C
- removed C117, C124, C50, C52, C59, C63: 0.1uF, Capacitor_SMD:C_0402_1005Metric, symbol Device:C
- removed C118, C119, C120, C121: 10nF, Capacitor_SMD:C_0603_1608Metric, symbol Device:C
- removed C46, C47, C56, C57: 82nF, Capacitor_SMD:C_0603_1608Metric, symbol PCM_Capacitor_AKL:C_Rect_L4.0mm_W2.5mm_P2.50mm
- removed C48, C49, C64, C65: 5.6nF, Capacitor_SMD:C_0603_1608Metric, symbol PCM_Capacitor_AKL:C_Rect_L4.0mm_W2.5mm_P2.50mm
- removed C66, C68, C69, C70, C71: 1uF, Capacitor_SMD:C_0402_1005Metric, symbol Device:C
- removed C74: 10nF, Capacitor_SMD:C_0402_1005Metric, symbol Device:C
- removed C78, C97, C99: 100nF, Capacitor_SMD:C_0402_1005Metric, symbol Device:C
- removed C85, C87: 1nF, Capacitor_SMD:C_0402_1005Metric, symbol Device:C
- removed C89, C90, C91, C92: 220nF, Capacitor_SMD:C_0402_1005Metric, symbol Device:C
- removed J7, J8: Conn_01x02_Socket, lcsc:CONN-TH_2P-P5.00_WJ500V-5.08-2P, symbol Connector:Conn_01x02_Socket
- removed L1, L2, L3, L4: 10uH, lcsc:IND-SMD_L11.0-W10.5_SL1050-330M, symbol Device:L
- removed R12, R13, R14, R15, R21, R25, R30, R34: 10K, Resistor_SMD:R_0402_1005Metric, symbol Device:R
- removed R40: 47k, Resistor_SMD:R_0402_1005Metric, symbol Device:R
- removed R41: 75k, Resistor_SMD:R_0402_1005Metric, symbol Device:R
- removed R44, R45, R50: 100k, Resistor_SMD:R_0402_1005Metric, symbol Device:R
- removed R47, R48, R53, R70, R71, R72: 6K, Resistor_SMD:R_0402_1005Metric, symbol Device:R
- removed R51: 10k, Resistor_SMD:R_0402_1005Metric, symbol Device:R
- removed R64, R65, R66, R67: 3.3, Resistor_SMD:R_0402_1005Metric, symbol Device:R
- removed U16, U23, U7: NE5532DR, lcsc:SOIC-8_L4.9-W3.9-P1.27-LS6.0-BL, symbol lcsc:NE5532DR
- removed U18: TPA3116D2DAD_C2865736, lcsc:HTSSOP-32_L11.0-W6.1-P0.65-LS8.1-BL, symbol lcsc:TPA3116D2DAD_C2865736
Connections:
- net SUB SUM BUFF is gone; now on net SPEAKER SUM BUFF: C72.2, R57.2
- net TWEET SUM BUFF N is gone; now on an unnamed net: U20.8 (OUT1)
- net /SD TWEET/WOOF is gone; now on net MUTE SUB: VQ1.67 (PE14)
- net +3.3V: now also J6.6 (Pin_6); no longer J10.5 (Pin_5)
- net +5V: now also J10.5 (Pin_5); no longer J6.6 (Pin_6)
- net GND: now also U20.6 (IN1+)
- net MUTE SUB: no longer VQ1.140 (PB9)
- net /SD SUB: now also VQ1.76 (PB15); no longer VQ1.141 (PE0)
- net MUTE TWEET/WOOF: no longer names the net of VQ1.78 (PD9)
- net SS XRES GPIO: no longer names the net of U21.24 (~{XRES})
- net SS XRES GPIO: no longer VQ1.76 (PB15)
- net SUB AMP N renamed AMP N
- net SUB AMP P renamed AMP P
- net SUB SUM BUFF N renamed SPEAKER SUM BUFF N
- no-connect marks 93 -> 97
Other:
- moved on the sheet: C100, C102, C104, C109, C110, C115, C116, C122, C123, C67, C72, C73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
