File: hardware/om-god.kicad_sch (KiCad schematic)
At the start: 478 parts, among them CN1 DIN-504B-M10, CN2 DIN-504B-M10, J1 PJ-625G, J10 Conn_01x08_Pin, J11 Conn_01x02_Socket, J2 PJ-625G, J3 Conn_01x13_Pin, J4 Conn_01x03_Pin, J5 PJ-625G, J6 Conn_01x08_Pin, J9 Conn_01x02_Socket, Q1 Si7617DN, Q2 Si7617DN, Q3 Si7617DN, SW1 TS-1003ST-26, SW10 RotaryEncoder, SW11 TS-1003ST-26, SW12 TS-1003ST-26, SW13 TS-1003ST-26, SW14 TS-1003ST-26, SW15 TS-1003ST-26, SW16 TS-1003ST-26, SW17 TS-1003ST-26, SW18 TS-1003ST-26, SW19 RotaryEncoder, SW2 TS-1003ST-26, SW20 RotaryEncoder, SW21 TS-1003ST-26, SW22 TS-1003ST-26, SW23 TS-1003ST-26, SW24 TS-1003ST-26, SW25 TS-1003ST-26, SW26 TS-1003ST-26, SW27 TS-1003ST-26, SW28 TS-1003ST-26, SW29 TS-1003ST-26, SW3 TS-1003ST-26, SW30 TS-1003ST-26, SW31 TS-1003ST-26, SW32 TS-1003ST-26, SW33 RotaryEncoder, SW34 RotaryEncoder, SW35 TS-1003ST-26, SW36 TS-1003ST-26, SW37 TS-1003ST-26, SW38 TS-1003ST-26, SW39 TS-1003ST-26, SW4 TS-1003ST-26, SW40 TS-1003ST-26, SW41 TS-1003ST-26, SW42 TS-1003ST-26, SW43 TS-1003ST-26, SW44 TS-1003ST-26, SW45 TS-1003ST-26, SW46 TS-1003ST-26, SW47 TS-1003ST-26, SW48 TS-1003ST-26, SW49 TS-1003ST-26, SW5 RotaryEncoder, SW50 TS-1003ST-26, SW51 TS-1003ST-26, SW52 TS-1003ST-26, SW53 TS-1003ST-26, SW54 TS-1003ST-26, SW55 TS-1003ST-26, SW56 TS-1003ST-26, SW57 TS-1003ST-26, SW58 SW_Push, SW6 TS-1003ST-26, SW60 SW_Push, SW61 RotaryEncoder_Switch, SW7 TS-1003ST-26, SW8 TS-1003ST-26, SW9 TS-1003ST-26, U1 PCM5122PW, U11 NE5532DR, U15 TS5A23159RSER, U17 TPA6120A2DWP, U19 TPA3116D2DAD_C2865736, U2 PCM5122PW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

Commit message: h
Parts:
- removed C79, C84: 0.1uF, Capacitor_SMD:C_0402_1005Metric, symbol Device:C
- removed R55, R56, R57: 6K, Resistor_SMD:R_0402_1005Metric, symbol Device:R
- removed U20: NE5532DR, lcsc:SOIC-8_L4.9-W3.9-P1.27-LS6.0-BL, symbol lcsc:NE5532DR
- added R12, R13, R14: 6K, Resistor_SMD:R_0402_1005Metric, symbol Device:R
Connections:
- net GND: now also R12.2; no longer U4.4 (IN2+)
- net SPEAKER SUM BUFF: now also R14.2
- net SPEAKER SUM BUFF N: now also U4.2 (OUT2), R13.1
- net at U4.3 (IN2-): now also R13.2, R14.1; no longer U4.2 (OUT2)
- new net: R12.1, U4.4 (IN2+)
Other:
- note added: "-12V Inverter"
- note added: "12V Bucker"
- note added: "3V3 BATT Bucker"
- note added: "3V3 Bucker"
- note added: "5V Bucker"
- note added: "Audio Processing"
- note added: "BATT Connector"
- note added: "Headphones"
- note added: "Midi"
- note added: "Midi In"
- note added: "Midi Out"
- note added: "Power Connector"
- note added: "Power Connetor"
- note added: "SD Card In"
- note added: "Speaker"
- note added: "Storage"
- note added: "Touch Pad"
- note added: "USB Type-C"
- moved on the sheet: AUDIO1, C1, C10, C100, C102, C104, C109, C11, C110, C115, C116, C12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
